File: hat/hat.sch (KiCad schematic (older format))
At the start: 4 parts

Commit message: made some connections
Parts:
- added J?: 52840 rx rpi tx, symbol Connector:Conn_01x02_Male
- added J?: 52840 tx pri rx, symbol Connector:Conn_01x02_Male
- added J?: sck, symbol Connector:Conn_01x02_Male
- added J?: mosi, symbol Connector:Conn_01x02_Male
- added J?: miso, symbol Connector:Conn_01x02_Male
- added J?: ss1, symbol Connector:Conn_01x02_Male
- added J?: nfc, symbol Connector:Conn_01x02_Male
- J?: value Conn_ARM_JTAG_SWD_10 -> 52840 swd
Connections:
- wire segments 4 -> 25
Changed lines of the file:
@@
 EESchema Schematic File Version 4
+LIBS:hat-cache
 EELAYER 26 0
 EELAYER END
@@
 L MCU_Nordic:nRF52840 U?
 U 1 1 5C1EABD8
-P 2550 3650
-F 0 "U?" H 2550 764 50  0000 C CNN
-F 1 "nRF52840" H 2550 673 50  0000 C CNN
-F 2 "Package_DFN_QFN:Nordic_AQFN-73-1EP_7x7mm_P0.5mm" H 2550 750 50  0001 C CNN
-F 3 "http://infocenter.nordicsemi.com/topic/com.nordic.infocenter.nrf52/dita/nrf52/chips/nrf52840.html" H 1900 5550 50  0001 C CNN
-	1    2550 3650
+P 3150 3650
+F 0 "U?" H 3150 764 50  0000 C CNN
+F 1 "nRF52840" H 3150 673 50  0000 C CNN
+F 2 "Package_DFN_QFN:Nordic_AQFN-73-1EP_7x7mm_P0.5mm" H 3150 750 50  0001 C CNN
+F 3 "http://infocenter.nordicsemi.com/topic/com.nordic.infocenter.nrf52/dita/nrf52/chips/nrf52840.html" H 2500 5550 50  0001 C CNN
+	1    3150 3650
 	1    0    0    -1
 $EndComp
@@
 	-1   0    0    1
 $EndComp
-Wire Wire Line
-	1350 1400 1350 1600
-Wire Wire Line
-	1350 1600 1150 1600
-Wire Wire Line
-	1150 1600 1150 1850
-Wire Wire Line
-	1150 1850 1250 1850
 $Comp
 L Connector:Raspberry_Pi_2_3 J?
@@
 L Connector:Conn_ARM_JTAG_SWD_10 J?
 U 1 1 5C1F1912
-P 5550 1400
-F 0 "J?" H 5110 1446 50  0000 R CNN
-F 1 "Conn_ARM_JTAG_SWD_10" H 5110 1355 50  0000 R CNN
-F 2 "Connector_PinHeader_1.27mm:PinHeader_2x05_P1.27mm_Vertical_SMD" H 5600 850 50  0001 L TNN
-F 3 "http://infocenter.arm.com/help/topic/com.arm.doc.faqs/attached/13634/cortex_debug_connectors.pdf" V 5200 150 50  0001 C CNN
-	1    5550 1400
+P 1250 6900
+F 0 "J?" H 810 6946 50  0000 R CNN
+F 1 "52840 swd" H 810 6855 50  0000 R CNN
+F 2 "Connector_PinHeader_1.27mm:PinHeader_2x05_P1.27mm_Vertical_SMD" H 1300 6350 50  0001 L TNN
+F 3 "http://infocenter.arm.com/help/topic/com.arm.doc.faqs/attached/13634/cortex_debug_connectors.pdf" V 900 5650 50  0001 C CNN
+	1    1250 6900
 	1    0    0    -1
 $EndComp
+$Comp
+L Connector:Conn_01x02_Male J?
+U 1 1 5C3A2B9D
+P 7600 3700
+F 0 "J?" H 7706 3878 50  0000 C CNN
+F 1 "52840 rx rpi tx" H 7706 3787 50  0000 C CNN
+F 2 "" H 7600 3700 50  0001 C CNN
+F 3 "~" H 7600 3700 50  0001 C CNN
+	1    7600 3700
+	1    0    0    -1
+$EndComp
+$Comp
+L Connector:Conn_01x02_Male J?
+U 1 1 5C3A2C4F
+P 7600 4050
+F 0 "J?" H 7706 4228 50  0000 C CNN
+F 1 "52840 tx pri rx" H 7706 4137 50  0000 C CNN
+F 2 "" H 7600 4050 50  0001 C CNN
+F 3 "~" H 7600 4050 50  0001 C CNN
+	1    7600 4050
+	1    0    0    -1
+$EndComp
+$Comp
+L Connector:Conn_01x02_Male J?
+U 1 1 5C3A387B
+P 7600 4650
+F 0 "J?" H 7706 4828 50  0000 C CNN
+F 1 "sck" H 7706 4737 50  0000 C CNN
+F 2 "" H 7600 4650 50  0001 C CNN
+F 3 "~" H 7600 4650 50  0001 C CNN
+	1    7600 4650
+	1    0    0    -1
+$EndComp
+$Comp
+L Connector:Conn_01x02_Male J?
+U 1 1 5C3A3882
+P 7600 5000
+F 0 "J?" H 7706 5178 50  0000 C CNN
+F 1 "mosi" H 7706 5087 50  0000 C CNN
+F 2 "" H 7600 5000 50  0001 C CNN
+F 3 "~" H 7600 5000 50  0001 C CNN
+	1    7600 5000
+	1    0    0    -1
+$EndComp
+$Comp
+L Connector:Conn_01x02_Male J?
+U 1 1 5C3A38EB
+P 7600 5400
+F 0 "J?" H 7706 5578 50  0000 C CNN
+F 1 "miso" H 7706 5487 50  0000 C CNN
+F 2 "" H 7600 5400 50  0001 C CNN
+F 3 "~" H 7600 5400 50  0001 C CNN
+	1    7600 5400
+	1    0    0    -1
+$EndComp
+$Comp
+L Connector:Conn_01x02_Male J?
+U 1 1 5C3A38F2
+P 7600 5750
+F 0 "J?" H 7706 5928 50  0000 C CNN
+F 1 "ss1" H 7706 5837 50  0000 C CNN
+F 2 "" H 7600 5750 50  0001 C CNN
+F 3 "~" H 7600 5750 50  0001 C CNN
+	1    7600 5750
+	1    0    0    -1
+$EndComp
+Wire Wire Line
+	7800 4850 7800 4750
+Wire Wire Line
+	9750 2600 9950 2600
+Wire Wire Line
+	9950 2600 9950 4650
+Wire Wire Line
+	9950 4650 7800 4650
+$Comp
+L Connector:Conn_01x02_Male J?
+U 1 1 5C3A8360
+P 5000 2150
+F 0 "J?" H 4972 2030 50  0000 R CNN
+F 1 "nfc " H 4972 2121 50  0000 R CNN
+F 2 "" H 5000 2150 50  0001 C CNN
+F 3 "~" H 5000 2150 50  0001 C CNN
+	1    5000 2150
+	-1   0    0    1
+$EndComp
+Wire Wire Line
+	1350 1400 1350 1850
+Wire Wire Line
+	1350 1850 1850 1850
+Wire Wire Line
+	4450 2050 4800 2050
+Wire Wire Line
+	4800 2150 4450 2150
+Wire Wire Line
+	4450 2950 6500 2950
+Wire Wire Line
+	7800 4850 6500 4850
+Wire Wire Line
+	6500 4850 6500 2950
+Wire Wire Line
+	1750 6600 1750 6150
+Wire Wire Line
+	1750 6150 1500 6150
+Wire Wire Line
+	1500 6150 1500 5350
+Wire Wire Line
+	1500 5350 1850 5350
+Wire Wire Line
+	1750 6800 1800 6800
+Wire Wire Line
+	1800 6800 1800 6100
+Wire Wire Line
+	1800 6100 1550 6100
+Wire Wire Line
+	1550 6100 1550 5450
+Wire Wire Line
+	1550 5450 1850 5450
+Wire Wire Line
+	1750 6900 1850 6900
+Wire Wire Line
+	1850 6900 1850 6050
+Wire Wire Line
+	1850 6050 1600 6050
+Wire Wire Line
+	1600 6050 1600 5550
+Wire Wire Line
+	1600 5550 1850 5550
 $EndSCHEMATC

Commit message: minor update
added datasheet
Connections:
- wire segments 25 -> 39
Changed lines of the file:
@@
-$Comp
-L Connector:Conn_01x02_Male J?
-U 1 1 5C3A2B9D
-P 7600 3700
-F 0 "J?" H 7706 3878 50  0000 C CNN
-F 1 "52840 rx rpi tx" H 7706 3787 50  0000 C CNN
-F 2 "" H 7600 3700 50  0001 C CNN
-F 3 "~" H 7600 3700 50  0001 C CNN
-	1    7600 3700
-	1    0    0    -1
-$EndComp
-$Comp
-L Connector:Conn_01x02_Male J?
-U 1 1 5C3A2C4F
-P 7600 4050
-F 0 "J?" H 7706 4228 50  0000 C CNN
-F 1 "52840 tx pri rx" H 7706 4137 50  0000 C CNN
-F 2 "" H 7600 4050 50  0001 C CNN
-F 3 "~" H 7600 4050 50  0001 C CNN
-	1    7600 4050
-	1    0    0    -1
-$EndComp
-$Comp
-L Connector:Conn_01x02_Male J?
-U 1 1 5C3A387B
-P 7600 4650
-F 0 "J?" H 7706 4828 50  0000 C CNN
-F 1 "sck" H 7706 4737 50  0000 C CNN
-F 2 "" H 7600 4650 50  0001 C CNN
-F 3 "~" H 7600 4650 50  0001 C CNN
-	1    7600 4650
-	1    0    0    -1
-$EndComp
-$Comp
-L Connector:Conn_01x02_Male J?
-U 1 1 5C3A3882
-P 7600 5000
-F 0 "J?" H 7706 5178 50  0000 C CNN
-F 1 "mosi" H 7706 5087 50  0000 C CNN
-F 2 "" H 7600 5000 50  0001 C CNN
-F 3 "~" H 7600 5000 50  0001 C CNN
-	1    7600 5000
-	1    0    0    -1
-$EndComp
-$Comp
-L Connector:Conn_01x02_Male J?
-U 1 1 5C3A38EB
-P 7600 5400
-F 0 "J?" H 7706 5578 50  0000 C CNN
-F 1 "miso" H 7706 5487 50  0000 C CNN
-F 2 "" H 7600 5400 50  0001 C CNN
-F 3 "~" H 7600 5400 50  0001 C CNN
-	1    7600 5400
-	1    0    0    -1
-$EndComp
-$Comp
-L Connector:Conn_01x02_Male J?
-U 1 1 5C3A38F2
-P 7600 5750
-F 0 "J?" H 7706 5928 50  0000 C CNN
-F 1 "ss1" H 7706 5837 50  0000 C CNN
-F 2 "" H 7600 5750 50  0001 C CNN
-F 3 "~" H 7600 5750 50  0001 C CNN
-	1    7600 5750
-	1    0    0    -1
-$EndComp
-Wire Wire Line
-	7800 4850 7800 4750
-Wire Wire Line
-	9750 2600 9950 2600
-Wire Wire Line
-	9950 2600 9950 4650
-Wire Wire Line
-	9950 4650 7800 4650
 $Comp
 L Connector:Conn_01x02_Male J?
@@
 Wire Wire Line
 	4800 2150 4450 2150
-Wire Wire Line
-	4450 2950 6500 2950
-Wire Wire Line
-	7800 4850 6500 4850
-Wire Wire Line
-	6500 4850 6500 2950
 Wire Wire Line
 	1750 6600 1750 6150
@@
 Wire Wire Line
 	1600 5550 1850 5550
+Wire Wire Line
+	6500 4850 6500 2950
+Wire Wire Line
+	4450 2950 6500 2950
+Wire Wire Line
+	9750 2600 9950 2600
+Wire Wire Line
+	9950 2600 9950 4650
+Wire Wire Line
+	7800 4850 6500 4850
+Wire Wire Line
+	9950 4650 7800 4650
+Wire Wire Line
+	7800 4850 7800 4750
+$Comp
+L Connector:Conn_01x02_Male J?
+U 1 1 5C3A38F2
+P 7600 5750
+F 0 "J?" H 7706 5928 50  0000 C CNN
+F 1 "ss1" H 7706 5837 50  0000 C CNN
+F 2 "" H 7600 5750 50  0001 C CNN
+F 3 "~" H 7600 5750 50  0001 C CNN
+	1    7600 5750
+	1    0    0    -1
+$EndComp
+$Comp
+L Connector:Conn_01x02_Male J?
+U 1 1 5C3A38EB
+P 7600 5400
+F 0 "J?" H 7706 5578 50  0000 C CNN
+F 1 "miso" H 7706 5487 50  0000 C CNN
+F 2 "" H 7600 5400 50  0001 C CNN
+F 3 "~" H 7600 5400 50  0001 C CNN
+	1    7600 5400
+	1    0    0    -1
+$EndComp
+$Comp
+L Connector:Conn_01x02_Male J?
+U 1 1 5C3A3882
+P 7600 5000
+F 0 "J?" H 7706 5178 50  0000 C CNN
+F 1 "mosi" H 7706 5087 50  0000 C CNN
+F 2 "" H 7600 5000 50  0001 C CNN
+F 3 "~" H 7600 5000 50  0001 C CNN
+	1    7600 5000
+	1    0    0    -1
+$EndComp
+$Comp
+L Connector:Conn_01x02_Male J?
+U 1 1 5C3A387B
+P 7600 4650
+F 0 "J?" H 7706 4828 50  0000 C CNN
+F 1 "sck" H 7706 4737 50  0000 C CNN
+F 2 "" H 7600 4650 50  0001 C CNN
+F 3 "~" H 7600 4650 50  0001 C CNN
+	1    7600 4650
+	1    0    0    -1
+$EndComp
+$Comp
+L Connector:Conn_01x02_Male J?
+U 1 1 5C3A2C4F
+P 5950 900
+F 0 "J?" H 6056 1078 50  0000 C CNN
+F 1 "52840 tx pri rx" H 6056 987 50  0000 C CNN
+F 2 "" H 5950 900 50  0001 C CNN
+F 3 "~" H 5950 900 50  0001 C CNN
+	1    5950 900
+	0    1    1    0
+$EndComp
+$Comp
+L Connector:Conn_01x02_Male J?
+U 1 1 5C3A2B9D
+P 6400 900
+F 0 "J?" H 6506 1078 50  0000 C CNN
+F 1 "52840 rx rpi tx" H 6506 987 50  0000 C CNN
+F 2 "" H 6400 900 50  0001 C CNN
+F 3 "~" H 6400 900 50  0001 C CNN
+	1    6400 900
+	0    1    1    0
+$EndComp
+Wire Wire Line
+	4450 1150 5850 1150
+Wire Wire Line
+	5850 1150 5850 1100
+Wire Wire Line
+	5950 1100 5950 1450
+Wire Wire Line
+	5950 1450 7100 1450
+Wire Wire Line
+	7100 1450 7100 1300
+Wire Wire Line
+	7100 1300 8150 1300
+Wire Wire Line
+	6400 1100 6400 1350
+Wire Wire Line
+	6400 1350 7000 1350
+Wire Wire Line
+	7000 1350 7000 1200
+Wire Wire Line
+	7000 1200 8150 1200
+Wire Wire Line
+	6300 1100 6300 1400
+Wire Wire Line
+	6300 1400 5750 1400
+Wire Wire Line
+	5750 1400 5750 1250
+Wire Wire Line
+	5750 1250 4450 1250
 $EndSCHEMATC

Commit message: placed labels and connectors
Parts:
- removed J?: sck, symbol Connector:Conn_01x02_Male
- removed J?: mosi, symbol Connector:Conn_01x02_Male
- removed J?: miso, symbol Connector:Conn_01x02_Male
- removed J?: ss1, symbol Connector:Conn_01x02_Male
- added J? (x2): Conn_02x20_Odd_Even, symbol Connector_Generic:Conn_02x20_Odd_Even
Connections:
- net labels added: P0.01, P0.02, P0.03, P0.04, P0.05, P0.06, P0.07, P0.08, P0.09, P0.10, P0.11, P0.12, P0.13, P0.14, P0.15, P0.16, P0.17, P0.18, P0.19, P0.20, P0.21, P0.22, P0.23, P0.24, P0.25, P0.26, P0.27, P0.28, P0.29, P0.30, p0.00
- wire segments 39 -> 99

Commit message: even more connectors added
added a ton of labels
Parts:
- removed J?: Conn_02x20_Odd_Even, symbol Connector_Generic:Conn_02x20_Odd_Even
- added J?: USB_A, symbol Connector:USB_A
- added P1: Conn_02x08_Odd_Even, symbol Connector_Generic:Conn_02x08_Odd_Even
- added Y?: 32mhzCrystal, symbol Device:Crystal
- gave numbers to parts that had none: 3
Connections:
- net labels added: 1.1vsup_decup, 1.3vsup_decup, 1.3vsup_decup(flash), 1.3vsup_decup(rf), 1.3vsup_decup2(rf), DCC, DCCH, Ground (Radio supply), P1.00, P1.01, P1.02, P1.03, P1.04, P1.05, P1.06, P1.07, P1.08, P1.09, P1.10, P1.11, P1.12, P1.13, P1.14, P1.15, VDD, VDDH, Vbus, XC1, XC2, decusb3.3v, psu_decup
- wire segments 99 -> 176
Other:
- note added: "_n____n__\n / \---||--<\n /___________\\n _|____|____|_\n _|____|____|_\n | | |\n --------------\n | || || || ||\\n | || || || || \++++++++------<\n ===============\n | | | | |\n (| O | O| O| O |)\n | | | | |\n (| O | O | O | O |)\n | | | | |\n (| O | O | O | O |)\n | | | | |\n (| O | O | O | O |)\n ======================"

Commit message: worked on schematic
added components
Parts:
- removed J?: Conn_Coaxial, symbol Connector:Conn_Coaxial
- added C? (x2): 12pf, symbol Device:C_Small
Connections:
- net labels added: 1.1vsup_decup(dec1), 1.3vsup_decup(dec4), 1.3vsup_decup(flash)(dec5), 1.3vsup_decup(rf)(dec2), 1.3vsup_decup2(rf)(dec6), Earth, Ground (VSS_PA), P0.31, VDD(b1), VSS, ant, psu_decup(dec3)
- net labels removed: 1.1vsup_decup, 1.3vsup_decup, 1.3vsup_decup(flash), 1.3vsup_decup(rf), 1.3vsup_decup2(rf), Ground (Radio supply), VDD, psu_decup
- wire segments 176 -> 189

Commit message: added ups board files
Connections:
- wire segments 189 -> 191
Changed lines of the file:
@@
 EESchema Schematic File Version 4
-LIBS:hat-cache
 EELAYER 26 0
 EELAYER END
@@
 Wire Wire Line
 	1750 6150 1500 6150
-Wire Wire Line
-	1500 6150 1500 5350
 Wire Wire Line
 	1500 5350 1850 5350
@@
 	3150 6800 3100 6800
 Connection ~ 3150 6800
+Wire Wire Line
+	1550 5200 1500 5200
+Wire Wire Line
+	1500 5200 1500 5350
+Connection ~ 1500 5350
+Wire Wire Line
+	1500 5350 1500 6150
 $EndSCHEMATC

Commit message: updated part
nrf52840 part updated
Parts:
- removed C? (x2): 12pf, symbol Device:C_Small
- removed J?: 52840 swd, Connector_PinHeader_1.27mm:PinHeader_2x05_P1.27mm_Vertical_SMD, symbol Connector:Conn_ARM_JTAG_SWD_10
- removed J?: nfc, symbol Connector:Conn_01x02_Male
- removed J?: USB_A, symbol Connector:USB_A
- removed Y?: 32mhzCrystal, symbol Device:Crystal
- removed soc1: nRF52840, Package_DFN_QFN:Nordic_AQFN-73-1EP_7x7mm_P0.5mm, symbol MCU_Nordic:nRF52840
- added C? (x2): 12pf, symbol Device:C_Small
- added J?: nfc, symbol Connector:Conn_01x02_Male
- added U?: nRF52840-QIAA, symbol nrf52840-qiaa:nRF52840-QIAA
- added Y?: 32mhzCrystal, symbol Device:Crystal
Connections:
- net labels added: VDD(A14), VDD(A22), VDD(AD23), VDD(W1)
- wire segments 191 -> 158

Commit message: updated file name and added sheet
updated file name and added sheet
Parts:
- removed C? (x2): 12pf, symbol Device:C_Small
- removed J1: Raspberry_Pi_2_3, symbol Connector:Raspberry_Pi_2_3
- removed J?: 52840 rx rpi tx, symbol Connector:Conn_01x02_Male
- removed J?: 52840 tx pri rx, symbol Connector:Conn_01x02_Male
- removed J?: nfc, symbol Connector:Conn_01x02_Male
- removed P0: Conn_02x20_Odd_Even, symbol Connector_Generic:Conn_02x20_Odd_Even
- removed P1: Conn_02x08_Odd_Even, symbol Connector_Generic:Conn_02x08_Odd_Even
- removed U?: nRF52840-QIAA, symbol nrf52840-qiaa:nRF52840-QIAA
- removed Y?: 32mhzCrystal, symbol Device:Crystal
Connections:
- net labels removed: 1.1vsup_decup(dec1), 1.3vsup_decup(dec4), 1.3vsup_decup(flash)(dec5), 1.3vsup_decup(rf)(dec2), 1.3vsup_decup2(rf)(dec6), DCC, DCCH, Earth, Ground (VSS_PA), P0.01, P0.02, P0.03, P0.04, P0.05, P0.06, P0.07, P0.08, P0.09, P0.10, P0.11, P0.12, P0.13, P0.14, P0.15, P0.16, P0.17, P0.18, P0.19, P0.20, P0.21, P0.22, P0.23, P0.24, P0.25, P0.26, P0.27, P0.28, P0.29, P0.30, P0.31, P1.00, P1.01, P1.02, P1.03, P1.04, P1.05, P1.06, P1.07, P1.08, P1.09, P1.10, P1.11, P1.12, P1.13, P1.14, P1.15, VDD(A14), VDD(A22), VDD(AD23), VDD(W1), VDD(b1), VDDH, VSS, Vbus, XC1, XC2, ant, decusb3.3v, p0.00, psu_decup(dec3)
- wire segments 158 -> 0
Other:
- note removed: "_n____n__\n / \---||--<\n /___________\\n _|____|____|_\n _|____|____|_\n | | |\n --------------\n | || || || ||\\n | || || || || \++++++++------<\n ===============\n | | | | |\n (| O | O| O| O |)\n | | | | |\n (| O | O | O | O |)\n | | | | |\n (| O | O | O | O |)\n | | | | |\n (| O | O | O | O |)\n ======================"
