File: hat/exturnal-power.sch (KiCad schematic (older format))
At the start: 9 parts

Commit message: fixed library stuff on main pc
please note that you will have to use the library loader to add all the right parts
Parts:
- removed IC?: LM2676S-5.0, TO127P1435X457-8N, symbol SamacSys_Parts:LM2676S-5.0
- added IC?: LM2676S-5.0, TO127P1435X457-8N, symbol SamacSys_Parts:LM2676S-5.0
Changed lines of the file:
@@
-$EndComp
-$Comp
-L SamacSys_Parts:LM2676S-5.0 IC?
-U 1 1 5C878082
-P 3500 1350
-F 0 "IC?" H 4150 1615 50  0000 C CNN
-F 1 "LM2676S-5.0" H 4150 1524 50  0000 C CNN
-F 2 "TO127P1435X457-8N" H 4650 1450 50  0001 L CNN
-F 3 "" H 4650 1350 50  0001 L CNN
-F 4 "IC BUCK 5V 3A" H 4650 1250 50  0001 L CNN "Description"
-F 5 "" H 4650 1150 50  0001 L CNN "Height"
-F 6 "926-LM2676S-50" H 4650 1050 50  0001 L CNN "Mouser Part Number"
-F 7 "https://www.mouser.com/Search/Refine.aspx?Keyword=926-LM2676S-50" H 4650 950 50  0001 L CNN "Mouser Price/Stock"
-F 8 "Texas Instruments" H 4650 850 50  0001 L CNN "Manufacturer_Name"
-F 9 "LM2676S-5.0" H 4650 750 50  0001 L CNN "Manufacturer_Part_Number"
-	1    3500 1350
-	1    0    0    -1
 $EndComp
 $Comp
@@
 Wire Wire Line
 	5350 1700 5600 1700
+$Comp
+L SamacSys_Parts:LM2676S-5.0 IC?
+U 1 1 5C7F86EF
+P 3500 1350
+F 0 "IC?" H 4150 1615 50  0000 C CNN
+F 1 "LM2676S-5.0" H 4150 1524 50  0000 C CNN
+F 2 "TO127P1435X457-8N" H 4650 1450 50  0001 L CNN
+F 3 "" H 4650 1350 50  0001 L CNN
+F 4 "IC BUCK 5V 3A" H 4650 1250 50  0001 L CNN "Description"
+F 5 "" H 4650 1150 50  0001 L CNN "Height"
+F 6 "926-LM2676S-50" H 4650 1050 50  0001 L CNN "Mouser Part Number"
+F 7 "https://www.mouser.com/Search/Refine.aspx?Keyword=926-LM2676S-50" H 4650 950 50  0001 L CNN "Mouser Price/Stock"
+F 8 "Texas Instruments" H 4650 850 50  0001 L CNN "Manufacturer_Name"
+F 9 "LM2676S-5.0" H 4650 750 50  0001 L CNN "Manufacturer_Part_Number"
+	1    3500 1350
+	1    0    0    -1
+$EndComp
 $EndSCHEMATC

Commit message: implemented the "ZVD" (or "ideal") diode
implements the "ZVD" (or "ideal") diode
reference https://github.com/raspberrypi/hats/blob/master/zvd-circuit.png
Parts:
- removed D?: ZVD, symbol pspice:DIODE
- added IC?: DMMT5401-7-F, SOT95P275X110-6N, symbol SamacSys_Parts:DMMT5401-7-F
- added Q?: DMG2305UX-7, SOT96P240X100-3N, symbol SamacSys_Parts:DMG2305UX-7
- added R?: 10k 1% 1005, symbol Device:R
- added R?: 47k 1% 1005, symbol Device:R
Connections:
- wire segments 40 -> 69
Changed lines of the file:
@@
 Comment4 ""
 $EndDescr
-Text GLabel 7500 1900 2    50   Input ~ 0
+Text GLabel 10100 1900 2    50   Input ~ 0
 rpi(5v)(pin2)
-Text GLabel 7500 1100 2    50   Input ~ 0
+Text GLabel 10100 1100 2    50   Input ~ 0
 rpi(GND)(pin6)
-$Comp
-L pspice:DIODE D?
-U 1 1 5C8775C8
-P 7150 1900
-F 0 "D?" H 7150 1635 50  0000 C CNN
-F 1 "ZVD" H 7150 1726 50  0000 C CNN
-F 2 "" H 7150 1900 50  0001 C CNN
-F 3 "" H 7150 1900 50  0001 C CNN
-	1    7150 1900
-	1    0    0    -1
-$EndComp
-Wire Wire Line
-	7350 1900 7500 1900
 $Comp
 L pspice:CAP C?
@@
 Wire Wire Line
 	6400 1700 6400 1800
-Wire Wire Line
-	6400 1700 6950 1700
-Wire Wire Line
-	6950 1700 6950 1900
 Connection ~ 6400 1700
 Wire Wire Line
@@
 	1    0    0    -1
 $EndComp
+$Comp
+L power:GNDREF #PWR?
+U 1 1 5C8067CD
+P 8050 2950
+F 0 "#PWR?" H 8050 2700 50  0001 C CNN
+F 1 "GNDREF" H 8055 2777 50  0000 C CNN
+F 2 "" H 8050 2950 50  0001 C CNN
+F 3 "" H 8050 2950 50  0001 C CNN
+	1    8050 2950
+	1    0    0    -1
+$EndComp
+$Comp
+L power:GNDREF #PWR?
+U 1 1 5C806E0E
+P 8450 2950
+F 0 "#PWR?" H 8450 2700 50  0001 C CNN
+F 1 "GNDREF" H 8455 2777 50  0000 C CNN
+F 2 "" H 8450 2950 50  0001 C CNN
+F 3 "" H 8450 2950 50  0001 C CNN
+	1    8450 2950
+	1    0    0    -1
+$EndComp
+Wire Wire Line
+	6400 2100 5600 2100
+Connection ~ 5600 2100
+$Comp
+L SamacSys_Parts:DMG2305UX-7 Q?
+U 1 1 5C807BC9
+P 8200 1200
+F 0 "Q?" V 8767 1300 50  0000 C CNN
+F 1 "DMG2305UX-7" V 8676 1300 50  0000 C CNN
+F 2 "SOT96P240X100-3N" H 8650 1150 50  0001 L CNN
+F 3 "https://componentsearchengine.com/Datasheets/1/DMG2305UX-7.pdf" H 8650 1050 50  0001 L CNN
+F 4 "MOSFET P-Ch 20V 5A Enhancement SOT23 Diodes Inc DMG2305UX-7 P-channel MOSFET Transistor, -3.3 A, -20 V, 3-Pin SOT-23" H 8650 950 50  0001 L CNN "Description"
+F 5 "1" H 8650 850 50  0001 L CNN "Height"
+F 6 "621-DMG2305UX-7" H 8650 750 50  0001 L CNN "Mouser Part Number"
+F 7 "https://www.mouser.com/Search/Refine.aspx?Keyword=621-DMG2305UX-7" H 8650 650 50  0001 L CNN "Mouser Price/Stock"
+F 8 "Diodes Inc." H 8650 550 50  0001 L CNN "Manufacturer_Name"
+F 9 "DMG2305UX-7" H 8650 450 50  0001 L CNN "Manufacturer_Part_Number"
+	1    8200 1200
+	0    -1   -1   0
+$EndComp
+$Comp
+L SamacSys_Parts:DMMT5401-7-F IC?
+U 1 1 5C807D70
+P 7600 2200
+F 0 "IC?" H 8050 2465 50  0000 C CNN
+F 1 "DMMT5401-7-F" H 8050 2374 50  0000 C CNN
+F 2 "SOT95P275X110-6N" H 8350 2300 50  0001 L CNN
+F 3 "https://componentsearchengine.com/Datasheets/1/DMMT5401-7-F.pdf" H 8350 2200 50  0001 L CNN
+F 4 "Transistor Dual PNP 150V 0.2A SOT26-6 Diodes Inc DMMT5401-7-F Dual PNP Bipolar Transistor, -200 mA, -150 V, 6-Pin SOT-26" H 8350 2100 50  0001 L CNN "Description"
+F 5 "1.1" H 8350 2000 50  0001 L CNN "Height"
+F 6 "621-DMMT5401-7-F" H 8350 1900 50  0001 L CNN "Mouser Part Number"
+F 7 "https://www.mouser.com/Search/Refine.aspx?Keyword=621-DMMT5401-7-F" H 8350 1800 50  0001 L CNN "Mouser Price/Stock"
+F 8 "Diodes Inc." H 8350 1700 50  0001 L CNN "Manufacturer_Name"
+F 9 "DMMT5401-7-F" H 8350 1600 50  0001 L CNN "Manufacturer_Part_Number"
+	1    7600 2200
+	0    -1   -1   0
+$EndComp
+$Comp
+L Device:R R?
+U 1 1 5C80BF79
+P 7700 2600
+F 0 "R?" H 7770 2646 50  0000 L CNN
+F 1 "10k 1% 1005" H 7770 2555 50  0000 L CNN
+F 2 "" V 7630 2600 50  0001 C CNN
+F 3 "~" H 7700 2600 50  0001 C CNN
+	1    7700 2600
+	1    0    0    -1
+$EndComp
+$Comp
+L Device:R R?
+U 1 1 5C80BFD7
+P 8450 2600
+F 0 "R?" H 8520 2646 50  0000 L CNN
+F 1 "47k 1% 1005" H 8520 2555 50  0000 L CNN
+F 2 "" V 8380 2600 50  0001 C CNN
+F 3 "~" H 8450 2600 50  0001 C CNN
+	1    8450 2600
+	1    0    0    -1
+$EndComp
+Wire Wire Line
+	6400 1700 6950 1700
+Wire Wire Line
+	6950 900  7800 900
+Wire Wire Line
+	7600 1300 6950 1300
+Wire Wire Line
+	6950 900  6950 1300
+Connection ~ 6950 1300
+Wire Wire Line
+	6950 1300 6950 1700
+Wire Wire Line
+	7700 1300 7700 1200
+Wire Wire Line
+	7700 1200 8000 1200
+Wire Wire Line
+	8000 1200 8000 1350
+Wire Wire Line
+	8000 1350 8650 1350
+Wire Wire Line
+	8650 1350 8650 900
+Wire Wire Line
+	8650 900  8400 900
+Wire Wire Line
+	7800 1300 7900 1300
+Wire Wire Line
+	7900 1300 7900 1450
+Wire Wire Line
+	7900 1450 8450 1450
+Wire Wire Line
+	8450 1450 8450 2200
+Wire Wire Line
+	8200 1200 8200 2200
+Wire Wire Line
+	8200 2200 8450 2200
+Connection ~ 8450 2200
+Wire Wire Line
+	8450 2200 8450 2450
+Wire Wire Line
+	7600 2200 7600 2350
+Wire Wire Line
+	7600 2350 7700 2350
+Wire Wire Line
+	7800 2350 7800 2200
+Wire Wire Line
+	7700 2200 7700 2350
+Connection ~ 7700 2350
+Wire Wire Line
+	7700 2350 7800 2350
+Wire Wire Line
+	7700 2350 7700 2450
+Wire Wire Line
+	7700 2750 7700 2850
+Wire Wire Line
+	7700 2850 8050 2850
+Wire Wire Line
+	8050 2850 8050 2950
+Wire Wire Line
+	8450 2750 8450 2950
+Wire Wire Line
+	8650 1350 9450 1350
+Wire Wire Line
+	9450 1350 9450 1900
+Wire Wire Line
+	9450 1900 10100 1900
+Connection ~ 8650 1350
 $EndSCHEMATC

Commit message: did stuff
Parts:
- added J?: Barrel_Jack, symbol Connector:Barrel_Jack
Connections:
- wire segments 69 -> 76
Other:
- note added: "nrf52840 and pi power"

Commit message: did some cleanup and added power connections
did some cleanup and added power connections
Connections:
- net labels added: VDD_HV, Vbus
- wire segments 76 -> 81
Changed lines of the file:
@@
 $EndComp
 $Comp
-L power:+12V #PWR?
+L power:+12V #PWR0118
 U 1 1 5C878161
 P 1100 4550
-F 0 "#PWR?" H 1100 4400 50  0001 C CNN
+F 0 "#PWR0118" H 1100 4400 50  0001 C CNN
 F 1 "+12V" H 1115 4723 50  0001 C CNN
 F 2 "" H 1100 4550 50  0001 C CNN
@@
 	3400 4750 3500 4750
 $Comp
-L power:GNDREF #PWR?
+L power:GNDREF #PWR0119
 U 1 1 5C87B557
 P 4050 5500
-F 0 "#PWR?" H 4050 5250 50  0001 C CNN
+F 0 "#PWR0119" H 4050 5250 50  0001 C CNN
 F 1 "GNDREF" H 4055 5327 50  0000 C CNN
 F 2 "" H 4050 5500 50  0001 C CNN
@@
 $EndComp
 $Comp
-L power:GNDREF #PWR?
+L power:GNDREF #PWR0120
 U 1 1 5C8067CD
 P 8050 6150
-F 0 "#PWR?" H 8050 5900 50  0001 C CNN
+F 0 "#PWR0120" H 8050 5900 50  0001 C CNN
 F 1 "GNDREF" H 8055 5977 50  0000 C CNN
 F 2 "" H 8050 6150 50  0001 C CNN
@@
 $EndComp
 $Comp
-L power:GNDREF #PWR?
+L power:GNDREF #PWR0121
 U 1 1 5C806E0E
 P 8450 6150
-F 0 "#PWR?" H 8450 5900 50  0001 C CNN
+F 0 "#PWR0121" H 8450 5900 50  0001 C CNN
 F 1 "GNDREF" H 8455 5977 50  0000 C CNN
 F 2 "" H 8450 6150 50  0001 C CNN
@@
 	3050 5500 3750 5500
 Wire Wire Line
-	8650 4550 10100 4550
+	8650 4550 10000 4550
 Wire Wire Line
 	2700 4100 2700 4300
@@
 Text Notes 5150 3750 0    79   ~ 0
 nrf52840 and pi power
+Text GLabel 10100 4750 2    50   Input ~ 0
+Vbus
+Wire Wire Line
+	10000 4550 10000 4650
+Wire Wire Line
+	10000 4750 10100 4750
+Connection ~ 10000 4550
+Wire Wire Line
+	10000 4550 10100 4550
+Wire Wire Line
+	10100 4650 10000 4650
+Connection ~ 10000 4650
+Wire Wire Line
+	10000 4650 10000 4750
+Text GLabel 10100 4650 2    50   Input ~ 0
+VDD_HV
 $EndSCHEMATC

Commit message: worked on power
Parts:
- removed J?: Barrel_Jack, symbol Connector:Barrel_Jack
- added J?: Screw_Terminal_01x02, symbol Connector:Screw_Terminal_01x02
Connections:
- net labels added: VSS_b7
- wire segments 81 -> 86
Changed lines of the file:
@@
 	8450 5950 8450 6150
 Connection ~ 8650 4550
-$Comp
-L Connector:Barrel_Jack J?
-U 1 1 5C7D5EA2
-P 1800 4000
-F 0 "J?" H 1855 4325 50  0000 C CNN
-F 1 "Barrel_Jack" H 1855 4234 50  0000 C CNN
-F 2 "" H 1850 3960 50  0001 C CNN
-F 3 "~" H 1850 3960 50  0001 C CNN
-	1    1800 4000
-	0    -1   1    0
-$EndComp
 Wire Wire Line
 	1100 4650 1700 4650
@@
 	2700 4100 2700 4300
 Connection ~ 2700 4300
-Wire Wire Line
-	2700 4300 1900 4300
 Wire Wire Line
 	2700 4100 2900 4100
@@
 Text GLabel 10100 4650 2    50   Input ~ 0
 VDD_HV
+Text GLabel 2900 3900 2    50   Input ~ 0
+VSS_b7
+$Comp
+L Connector:Screw_Terminal_01x02 J?
+U 1 1 5C9922FF
+P 1750 4000
+F 0 "J?" V 1716 3812 50  0000 R CNN
+F 1 "Screw_Terminal_01x02" V 1625 3812 50  0000 R CNN
+F 2 "" H 1750 4000 50  0001 C CNN
+F 3 "~" H 1750 4000 50  0001 C CNN
+	1    1750 4000
+	0    -1   -1   0
+$EndComp
+Wire Wire Line
+	1850 4300 1850 4200
+Wire Wire Line
+	1850 4300 2700 4300
+Wire Wire Line
+	1700 4300 1750 4300
+Wire Wire Line
+	1750 4300 1750 4200
+Wire Wire Line
+	2900 3900 2700 3900
+Wire Wire Line
+	2700 3900 2700 4100
+Connection ~ 2700 4100
 $EndSCHEMATC

Commit message: did some cleanup
Parts:
- added J?: Screw_Terminal_01x01, symbol Connector:Screw_Terminal_01x01
Connections:
- wire segments 86 -> 89
Changed lines of the file:
@@
 Wire Wire Line
 	3400 4750 3500 4750
-$Comp
-L power:GNDREF #PWR0119
-U 1 1 5C87B557
-P 4050 5500
-F 0 "#PWR0119" H 4050 5250 50  0001 C CNN
-F 1 "GNDREF" H 4055 5327 50  0000 C CNN
-F 2 "" H 4050 5500 50  0001 C CNN
-F 3 "" H 4050 5500 50  0001 C CNN
-	1    4050 5500
-	1    0    0    -1
-$EndComp
 Wire Wire Line
 	5600 5300 4050 5300
-Wire Wire Line
-	4050 5300 4050 5500
 Wire Wire Line
 	2450 5500 3050 5500
@@
 	1    0    0    -1
 $EndComp
-$Comp
-L power:GNDREF #PWR0120
-U 1 1 5C8067CD
-P 8050 6150
-F 0 "#PWR0120" H 8050 5900 50  0001 C CNN
-F 1 "GNDREF" H 8055 5977 50  0000 C CNN
-F 2 "" H 8050 6150 50  0001 C CNN
-F 3 "" H 8050 6150 50  0001 C CNN
-	1    8050 6150
-	1    0    0    -1
-$EndComp
-$Comp
-L power:GNDREF #PWR0121
-U 1 1 5C806E0E
-P 8450 6150
-F 0 "#PWR0121" H 8450 5900 50  0001 C CNN
-F 1 "GNDREF" H 8455 5977 50  0000 C CNN
-F 2 "" H 8450 6150 50  0001 C CNN
-F 3 "" H 8450 6150 50  0001 C CNN
-	1    8450 6150
-	1    0    0    -1
-$EndComp
 Wire Wire Line
 	6400 5300 5600 5300
@@
 	7700 5950 7700 6050
 Wire Wire Line
-	7700 6050 8050 6050
-Wire Wire Line
-	8050 6050 8050 6150
-Wire Wire Line
-	8450 5950 8450 6150
+	8450 5950 8450 6050
 Connection ~ 8650 4550
 Wire Wire Line
@@
 	2700 3900 2700 4100
 Connection ~ 2700 4100
+Wire Wire Line
+	7700 6050 6400 6050
+Wire Wire Line
+	6400 6050 6400 5300
+Connection ~ 7700 6050
+Connection ~ 6400 5300
+Wire Wire Line
+	7700 6050 8450 6050
+$Comp
+L power:GNDREF #PWR?
+U 1 1 5C85FDB7
+P 3050 5650
+F 0 "#PWR?" H 3050 5400 50  0001 C CNN
+F 1 "GNDREF" H 3055 5477 50  0000 C CNN
+F 2 "" H 3050 5650 50  0001 C CNN
+F 3 "" H 3050 5650 50  0001 C CNN
+	1    3050 5650
+	1    0    0    -1
+$EndComp
+Wire Wire Line
+	3050 5500 3050 5650
+$Comp
+L Connector:Screw_Terminal_01x01 J?
+U 1 1 5C86EF16
+P 4950 3750
+F 0 "J?" V 4916 3662 50  0000 R CNN
+F 1 "Screw_Terminal_01x01" V 4825 3662 50  0000 R CNN
+F 2 "" H 4950 3750 50  0001 C CNN
+F 3 "~" H 4950 3750 50  0001 C CNN
+	1    4950 3750
+	0    -1   -1   0
+$EndComp
+Wire Wire Line
+	4800 4750 4950 4750
+Wire Wire Line
+	4950 4750 4950 3950
 $EndSCHEMATC

Commit message: added sma connector
Connections:
- net labels added: Earth
- net labels removed: GNDREF
- wire segments 89 -> 90
Changed lines of the file:
@@
 Connection ~ 3050 5500
 Wire Wire Line
-	3050 5500 3750 5500
+	3050 5500 3400 5500
 Wire Wire Line
 	8650 4550 10000 4550
@@
 	7700 6050 8450 6050
 $Comp
-L power:GNDREF #PWR?
-U 1 1 5C85FDB7
-P 3050 5650
-F 0 "#PWR?" H 3050 5400 50  0001 C CNN
-F 1 "GNDREF" H 3055 5477 50  0000 C CNN
-F 2 "" H 3050 5650 50  0001 C CNN
-F 3 "" H 3050 5650 50  0001 C CNN
-	1    3050 5650
-	1    0    0    -1
-$EndComp
-Wire Wire Line
-	3050 5500 3050 5650
-$Comp
 L Connector:Screw_Terminal_01x01 J?
 U 1 1 5C86EF16
@@
 Wire Wire Line
 	4950 4750 4950 3950
+$Comp
+L power:Earth #PWR?
+U 1 1 5C86ED5A
+P 3400 5650
+F 0 "#PWR?" H 3400 5400 50  0001 C CNN
+F 1 "Earth" H 3400 5500 50  0001 C CNN
+F 2 "" H 3400 5650 50  0001 C CNN
+F 3 "~" H 3400 5650 50  0001 C CNN
+	1    3400 5650
+	1    0    0    -1
+$EndComp
+Wire Wire Line
+	3400 5650 3400 5500
+Connection ~ 3400 5500
+Wire Wire Line
+	3400 5500 3750 5500
 $EndSCHEMATC

Commit message: started pcb
Parts:
- C17, C18: renamed from C?; footprint (none) -> Capacitor_SMD:CP_Elec_3x5.4
- C19, C20: renamed from C?; footprint (none) -> Capacitor_SMD:C_0805_2012Metric_Pad1.15x1.40mm_HandSolder; symbol pspice:CAP -> Device:C
- C21: renamed from C?; footprint (none) -> Capacitor_SMD:CP_Elec_3x5.3
- D1: renamed from D?; footprint (none) -> Diode_SMD:D_0805_2012Metric_Pad1.15x1.40mm_HandSolder
- IC1: renamed from IC?; footprint TO127P1435X457-8N -> SamacSys_Parts:TO127P1435X457-8N
- IC2: renamed from IC?; footprint SOT95P275X110-6N -> SamacSys_Parts:SOT95P275X110-6N
- J7: renamed from J?; footprint (none) -> TerminalBlock:TerminalBlock_Altech_AK300-2_P5.00mm
- J8: renamed from J?; footprint (none) -> TerminalBlock_MetzConnect:TerminalBlock_MetzConnect_360271_1x01_Horizontal_ScrewM3.0_Boxed
- L5: renamed from L?; footprint (none) -> Inductor_SMD:L_0805_2012Metric_Pad1.15x1.40mm_HandSolder
- Q1: renamed from Q?; footprint SOT96P240X100-3N -> SamacSys_Parts:SOT96P240X100-3N
- R1, R2: renamed from R?; footprint (none) -> Resistor_SMD:R_0805_2012Metric_Pad1.15x1.40mm_HandSolder
Connections:
- wire segments 90 -> 92
Changed lines of the file:
@@
 rpi(GND)(pin6)
 $Comp
-L pspice:CAP C?
+L Device:C C19
 U 1 1 5C8776E3
 P 2450 5250
-F 0 "C?" H 2628 5296 50  0000 L CNN
+F 0 "C19" H 2628 5296 50  0000 L CNN
 F 1 "0.47uf" H 2628 5205 50  0000 L CNN
-F 2 "" H 2450 5250 50  0001 C CNN
+F 2 "Capacitor_SMD:C_0805_2012Metric_Pad1.15x1.40mm_HandSolder" H 2450 5250 50  0001 C CNN
 F 3 "" H 2450 5250 50  0001 C CNN
 	1    2450 5250
@@
 $EndComp
 $Comp
-L Device:CP1 C?
+L Device:CP1 C17
 U 1 1 5C877F34
 P 1100 5300
-F 0 "C?" H 1215 5346 50  0000 L CNN
+F 0 "C17" H 1215 5346 50  0000 L CNN
 F 1 "15uf/50v" H 1215 5255 50  0000 L CNN
-F 2 "" H 1100 5300 50  0001 C CNN
+F 2 "Capacitor_SMD:CP_Elec_3x5.4" H 1100 5300 50  0001 C CNN
 F 3 "~" H 1100 5300 50  0001 C CNN
 	1    1100 5300
@@
 $EndComp
 $Comp
-L Device:CP1 C?
+L Device:CP1 C18
 U 1 1 5C877FA6
 P 1750 5300
-F 0 "C?" H 1865 5346 50  0000 L CNN
+F 0 "C18" H 1865 5346 50  0000 L CNN
 F 1 "15uf/50v" H 1865 5255 50  0000 L CNN
-F 2 "" H 1750 5300 50  0001 C CNN
+F 2 "Capacitor_SMD:CP_Elec_3x5.4" H 1750 5300 50  0001 C CNN
 F 3 "~" H 1750 5300 50  0001 C CNN
 	1    1750 5300
@@
 $EndComp
 $Comp
-L Device:D_Schottky D?
+L Device:D_Schottky D1
 U 1 1 5C8798B5
 P 5600 5150
-F 0 "D?" V 5554 5229 50  0000 L CNN
+F 0 "D1" V 5554 5229 50  0000 L CNN
 F 1 "SR305" V 5645 5229 50  0000 L CNN
-F 2 "" H 5600 5150 50  0001 C CNN
+F 2 "Diode_SMD:D_0805_2012Metric_Pad1.15x1.40mm_HandSolder" H 5600 5150 50  0001 C CNN
 F 3 "~" H 5600 5150 50  0001 C CNN
 	1    5600 5150
@@
 $EndComp
 $Comp
-L pspice:CAP C?
+L Device:C C20
 U 1 1 5C87999F
 P 5600 4550
-F 0 "C?" H 5422 4504 50  0000 R CNN
+F 0 "C20" H 5422 4504 50  0000 R CNN
 F 1 "0.01uf" H 5422 4595 50  0000 R CNN
-F 2 "" H 5600 4550 50  0001 C CNN
+F 2 "Capacitor_SMD:C_0805_2012Metric_Pad1.15x1.40mm_HandSolder" H 5600 4550 50  0001 C CNN
 F 3 "" H 5600 4550 50  0001 C CNN
 	1    5600 4550
@@
 $EndComp
 $Comp
-L Device:L L?
+L Device:L L5
 U 1 1 5C87ADF0
 P 6200 4900
-F 0 "L?" V 6390 4900 50  0000 C CNN
+F 0 "L5" V 6390 4900 50  0000 C CNN
 F 1 "10uH" V 6299 4900 50  0000 C CNN
-F 2 "" H 6200 4900 50  0001 C CNN
+F 2 "Inductor_SMD:L_0805_2012Metric_Pad1.15x1.40mm_HandSolder" H 6200 4900 50  0001 C CNN
 F 3 "~" H 6200 4900 50  0001 C CNN
 	1    6200 4900
@@
 $EndComp
 $Comp
-L Device:CP1 C?
+L Device:CP1 C21
 U 1 1 5C87B06D
 P 6400 5150
-F 0 "C?" H 6515 5196 50  0000 L CNN
+F 0 "C21" H 6515 5196 50  0000 L CNN
 F 1 "180uf/16v" H 6515 5105 50  0000 L CNN
-F 2 "" H 6400 5150 50  0001 C CNN
+F 2 "Capacitor_SMD:CP_Elec_3x5.3" H 6400 5150 50  0001 C CNN
 F 3 "~" H 6400 5150 50  0001 C CNN
 	1    6400 5150
@@
 Wire Wire Line
 	5600 4900 5600 5000
-Wire Wire Line
-	5600 4800 5600 4900
 Connection ~ 5600 4900
 Wire Wire Line
@@
 Wire Wire Line
 	5600 5300 4050 5300
-Wire Wire Line
-	2450 5500 3050 5500
 Wire Wire Line
 	3750 5500 3750 5300
@@
 Connection ~ 4050 5300
 Wire Wire Line
-	2450 5500 1750 5500
-Wire Wire Line
 	1750 5500 1750 5450
-Connection ~ 2450 5500
 Wire Wire Line
 	1750 5500 1100 5500
@@
 Wire Wire Line
 	1100 4850 1750 4850
-Wire Wire Line
-	2450 4850 2450 5000
 Connection ~ 1100 4850
 Wire Wire Line
@@
 	5350 4900 5600 4900
 $Comp
-L SamacSys_Parts:LM2676S-5.0 IC?
+L SamacSys_Parts:LM2676S-5.0 IC1
 U 1 1 5C7F86EF
 P 3500 4550
-F 0 "IC?" H 4150 4815 50  0000 C CNN
+F 0 "IC1" H 4150 4815 50  0000 C CNN
 F 1 "LM2676S-5.0" H 4150 4724 50  0000 C CNN
-F 2 "TO127P1435X457-8N" H 4650 4650 50  0001 L CNN
+F 2 "SamacSys_Parts:TO127P1435X457-8N" H 4650 4650 50  0001 L CNN
 F 3 "" H 4650 4550 50  0001 L CNN
 F 4 "IC BUCK 5V 3A" H 4650 4450 50  0001 L CNN "Description"
@@
 Connection ~ 5600 5300
 $Comp
-L SamacSys_Parts:DMG2305UX-7 Q?
+L SamacSys_Parts:DMG2305UX-7 Q1
 U 1 1 5C807BC9
 P 8200 4400
-F 0 "Q?" V 8767 4500 50  0000 C CNN
+F 0 "Q1" V 8767 4500 50  0000 C CNN
 F 1 "DMG2305UX-7" V 8676 4500 50  0000 C CNN
-F 2 "SOT96P240X100-3N" H 8650 4350 50  0001 L CNN
+F 2 "SamacSys_Parts:SOT96P240X100-3N" H 8650 4350 50  0001 L CNN
 F 3 "https://componentsearchengine.com/Datasheets/1/DMG2305UX-7.pdf" H 8650 4250 50  0001 L CNN
 F 4 "MOSFET P-Ch 20V 5A Enhancement SOT23 Diodes Inc DMG2305UX-7 P-channel MOSFET Transistor, -3.3 A, -20 V, 3-Pin SOT-23" H 8650 4150 50  0001 L CNN "Description"
@@
 $EndComp
 $Comp
-L SamacSys_Parts:DMMT5401-7-F IC?
+L SamacSys_Parts:DMMT5401-7-F IC2
 U 1 1 5C807D70
 P 7600 5400
-F 0 "IC?" H 8050 5665 50  0000 C CNN
+F 0 "IC2" H 8050 5665 50  0000 C CNN
 F 1 "DMMT5401-7-F" H 8050 5574 50  0000 C CNN
-F 2 "SOT95P275X110-6N" H 8350 5500 50  0001 L CNN
+F 2 "SamacSys_Parts:SOT95P275X110-6N" H 8350 5500 50  0001 L CNN
 F 3 "https://componentsearchengine.com/Datasheets/1/DMMT5401-7-F.pdf" H 8350 5400 50  0001 L CNN
 F 4 "Transistor Dual PNP 150V 0.2A SOT26-6 Diodes Inc DMMT5401-7-F Dual PNP Bipolar Transistor, -200 mA, -150 V, 6-Pin SOT-26" H 8350 5300 50  0001 L CNN "Description"
@@
 $EndComp
 $Comp
-L Device:R R?
+L Device:R R1
 U 1 1 5C80BF79
 P 7700 5800
-F 0 "R?" H 7770 5846 50  0000 L CNN
+F 0 "R1" H 7770 5846 50  0000 L CNN
 F 1 "10k 1% 1005" H 7770 5755 50  0000 L CNN
-F 2 "" V 7630 5800 50  0001 C CNN
+F 2 "Resistor_SMD:R_0805_2012Metric_Pad1.15x1.40mm_HandSolder" V 7630 5800 50  0001 C CNN
 F 3 "~" H 7700 5800 50  0001 C CNN
 	1    7700 5800
@@
 $EndComp
 $Comp
-L Device:R R?
+L Device:R R2
 U 1 1 5C80BFD7
 P 8450 5800
-F 0 "R?" H 8520 5846 50  0000 L CNN
+F 0 "R2" H 8520 5846 50  0000 L CNN
 F 1 "47k 1% 1005" H 8520 5755 50  0000 L CNN
-F 2 "" V 8380 5800 50  0001 C CNN
+F 2 "Resistor_SMD:R_0805_2012Metric_Pad1.15x1.40mm_HandSolder" V 8380 5800 50  0001 C CNN
 F 3 "~" H 8450 5800 50  0001 C CNN
 	1    8450 5800
@@
 VSS_b7
 $Comp
-L Connector:Screw_Terminal_01x02 J?
+L Connector:Screw_Terminal_01x02 J7
 U 1 1 5C9922FF
 P 1750 4000
-F 0 "J?" V 1716 3812 50  0000 R CNN
+F 0 "J7" V 1716 3812 50  0000 R CNN
 F 1 "Screw_Terminal_01x02" V 1625 3812 50  0000 R CNN
-F 2 "" H 1750 4000 50  0001 C CNN
+F 2 "TerminalBlock:TerminalBlock_Altech_AK300-2_P5.00mm" H 1750 4000 50  0001 C CNN
 F 3 "~" H 1750 4000 50  0001 C CNN
 	1    1750 4000
@@
 	7700 6050 8450 6050
 $Comp
-L Connector:Screw_Terminal_01x01 J?
+L Connector:Screw_Terminal_01x01 J8
 U 1 1 5C86EF16
 P 4950 3750
-F 0 "J?" V 4916 3662 50  0000 R CNN
+F 0 "J8" V 4916 3662 50  0000 R CNN
 F 1 "Screw_Terminal_01x01" V 4825 3662 50  0000 R CNN
-F 2 "" H 4950 3750 50  0001 C CNN
+F 2 "TerminalBlock_MetzConnect:TerminalBlock_MetzConnect_360271_1x01_Horizontal_ScrewM3.0_Boxed" H 4950 3750 50  0001 C CNN
 F 3 "~" H 4950 3750 50  0001 C CNN
 	1    4950 3750
@@
 	4950 4750 4950 3950
 $Comp
-L power:Earth #PWR?
+L power:Earth #PWR0105
 U 1 1 5C86ED5A
 P 3400 5650
-F 0 "#PWR?" H 3400 5400 50  0001 C CNN
+F 0 "#PWR0105" H 3400 5400 50  0001 C CNN
 F 1 "Earth" H 3400 5500 50  0001 C CNN
 F 2 "" H 3400 5650 50  0001 C CNN
@@
 Wire Wire Line
 	3400 5500 3750 5500
+Wire Wire Line
+	5600 4400 5600 4300
+Wire Wire Line
+	1750 5500 2450 5500
+Wire Wire Line
+	5600 4700 5600 4900
+Wire Wire Line
+	2450 5400 2450 5500
+Connection ~ 2450 5500
+Wire Wire Line
+	2450 5500 3050 5500
+Wire Wire Line
+	2450 4850 2450 5100
 $EndSCHEMATC
