File: hat/exturnal-power.sch (KiCad schematic (older format))
At the start: 14 parts, among them IC1 LM2676S-5.0, IC2 DMMT5401-7-F, J7 Screw_Terminal_01x02, J8 Screw_Terminal_01x01, Q1 DMG2305UX-7

Commit message: added basic varient
Parts:
- renumbered C17 to C18, C18 to C19, C19 to C20, C20 to C21, C21 to C22, L5 to L6
Changed lines of the file:
@@
 rpi(GND)(pin6)
 $Comp
-L Device:C C19
+L Device:C C20
 U 1 1 5C8776E3
 P 2450 5250
-F 0 "C19" H 2628 5296 50  0000 L CNN
+F 0 "C20" H 2628 5296 50  0000 L CNN
 F 1 "0.47uf" H 2628 5205 50  0000 L CNN
 F 2 "Capacitor_SMD:C_0805_2012Metric_Pad1.15x1.40mm_HandSolder" H 2450 5250 50  0001 C CNN
@@
 $EndComp
 $Comp
-L Device:CP1 C17
+L Device:CP1 C18
 U 1 1 5C877F34
 P 1100 5300
-F 0 "C17" H 1215 5346 50  0000 L CNN
+F 0 "C18" H 1215 5346 50  0000 L CNN
 F 1 "15uf/50v" H 1215 5255 50  0000 L CNN
 F 2 "Capacitor_SMD:CP_Elec_3x5.4" H 1100 5300 50  0001 C CNN
@@
 $EndComp
 $Comp
-L Device:CP1 C18
+L Device:CP1 C19
 U 1 1 5C877FA6
 P 1750 5300
-F 0 "C18" H 1865 5346 50  0000 L CNN
+F 0 "C19" H 1865 5346 50  0000 L CNN
 F 1 "15uf/50v" H 1865 5255 50  0000 L CNN
 F 2 "Capacitor_SMD:CP_Elec_3x5.4" H 1750 5300 50  0001 C CNN
@@
 $EndComp
 $Comp
-L power:+12V #PWR0118
+L power:+12V #PWR017
 U 1 1 5C878161
 P 1100 4550
-F 0 "#PWR0118" H 1100 4400 50  0001 C CNN
+F 0 "#PWR017" H 1100 4400 50  0001 C CNN
 F 1 "+12V" H 1115 4723 50  0001 C CNN
 F 2 "" H 1100 4550 50  0001 C CNN
@@
 $EndComp
 $Comp
-L Device:C C20
+L Device:C C21
 U 1 1 5C87999F
 P 5600 4550
-F 0 "C20" H 5422 4504 50  0000 R CNN
+F 0 "C21" H 5422 4504 50  0000 R CNN
 F 1 "0.01uf" H 5422 4595 50  0000 R CNN
 F 2 "Capacitor_SMD:C_0805_2012Metric_Pad1.15x1.40mm_HandSolder" H 5600 4550 50  0001 C CNN
@@
 $EndComp
 $Comp
-L Device:L L5
+L Device:L L6
 U 1 1 5C87ADF0
 P 6200 4900
-F 0 "L5" V 6390 4900 50  0000 C CNN
+F 0 "L6" V 6390 4900 50  0000 C CNN
 F 1 "10uH" V 6299 4900 50  0000 C CNN
 F 2 "Inductor_SMD:L_0805_2012Metric_Pad1.15x1.40mm_HandSolder" H 6200 4900 50  0001 C CNN
@@
 $EndComp
 $Comp
-L Device:CP1 C21
+L Device:CP1 C22
 U 1 1 5C87B06D
 P 6400 5150
-F 0 "C21" H 6515 5196 50  0000 L CNN
+F 0 "C22" H 6515 5196 50  0000 L CNN
 F 1 "180uf/16v" H 6515 5105 50  0000 L CNN
 F 2 "Capacitor_SMD:CP_Elec_3x5.3" H 6400 5150 50  0001 C CNN
@@
 	4950 4750 4950 3950
 $Comp
-L power:Earth #PWR0105
+L power:Earth #PWR018
 U 1 1 5C86ED5A
 P 3400 5650
-F 0 "#PWR0105" H 3400 5400 50  0001 C CNN
+F 0 "#PWR018" H 3400 5400 50  0001 C CNN
 F 1 "Earth" H 3400 5500 50  0001 C CNN
 F 2 "" H 3400 5650 50  0001 C CNN
