File: hat/nrf52840-and-connectors.sch (KiCad schematic (older format))
At the start: 20 parts

Commit message: started external power input schematic
-please note this is not edited to be right it just has all the parts added based off the diagram in the lm2676 datasheet 
-power link it rpi added
Connections:
- net labels added: rpi(5v)(pin2), rpi(GND)(pin6)
- wire segments 316 -> 320
Changed lines of the file:
@@
 $Descr A4 11693 8268
 encoding utf-8
-Sheet 3 3
+Sheet 3 4
 Title ""
 Date ""
@@
 AR Path="/5C9FDFE4/5CD8A302" Ref="#PWR?"  Part="1"
 AR Path="/5CD8A302" Ref="#PWR?"  Part="1"
+AR Path="/5CD5D522/5CD8A302" Ref="#PWR?"  Part="1"
 F 0 "#PWR?" H -10200 -2100 50  0001 C CNN
 F 1 "Earth" H -10200 -2000 50  0001 C CNN
@@
 AR Path="/5C9FDFE4/5CD957DC" Ref="#PWR?"  Part="1"
 AR Path="/5CD957DC" Ref="#PWR?"  Part="1"
+AR Path="/5CD5D522/5CD957DC" Ref="#PWR?"  Part="1"
 F 0 "#PWR?" H 700 5400 50  0001 C CNN
 F 1 "Earth" H 700 5500 50  0001 C CNN
@@
 Wire Wire Line
 	2100 1700 1950 1700
+Text GLabel 8100 750  0    50   Input ~ 0
+rpi(5v)(pin2)
+Text GLabel 8400 3550 0    50   Input ~ 0
+rpi(GND)(pin6)
+Wire Wire Line
+	8100 750  8750 750
+Wire Wire Line
+	8750 750  8750 800
+Wire Wire Line
+	8400 3550 8550 3550
+Wire Wire Line
+	8550 3550 8550 3400
 $EndSCHEMATC

Commit message: did some stuff tried to fix some things
did some stuff tried to fix some things nrf52840 part keeps disappearing
Parts:
- removed C? (x2): 12pf, symbol Device:C_Small
- removed J?: Raspberry_Pi_2_3, symbol Connector:Raspberry_Pi_2_3
- removed J?: 52840 tx pri rx, symbol Connector:Conn_01x02_Male
- removed J?: 52840 rx rpi tx, symbol Connector:Conn_01x02_Male
- removed J?: nfc, symbol Connector:Conn_01x02_Male
- removed P?: Conn_02x20_Odd_Even, symbol Connector_Generic:Conn_02x20_Odd_Even
- removed P?: Conn_02x08_Odd_Even, symbol Connector_Generic:Conn_02x08_Odd_Even
- removed U? (x2): nRF52840-QIAA, symbol nrf52840-qiaa:nRF52840-QIAA
- removed Y?: 32mhzCrystal, symbol Device:Crystal
Connections:
- wire segments 320 -> 162

Commit message: fixed library stuff on main pc
please note that you will have to use the library loader to add all the right parts
Parts:
- added U?: nRF52840-QIAA, symbol nrf52840-qiaa:nRF52840-QIAA
Changed lines of the file:
@@
 	-1   0    0    1
 $EndComp
-Wire Wire Line
-	4300 1400 5400 1400
-Wire Wire Line
-	4300 1300 5400 1300
 Text GLabel 5400 1200 0    50   Input ~ 0
 p0.00
@@
 	5400 1400 5600 1400
 Wire Wire Line
-	4500 1500 4300 1500
-Wire Wire Line
-	4300 1600 4500 1600
-Wire Wire Line
-	4500 1700 4300 1700
-Wire Wire Line
 	4300 1800 4500 1800
 Wire Wire Line
-	4500 1900 4300 1900
-Wire Wire Line
-	4500 2000 4300 2000
-Wire Wire Line
 	4300 2100 4500 2100
 Wire Wire Line
-	4500 2400 4300 2400
-Wire Wire Line
 	4300 2500 4500 2500
 Wire Wire Line
-	4500 2600 4300 2600
-Wire Wire Line
 	4300 2700 4500 2700
 Wire Wire Line
-	4500 2800 4300 2800
-Wire Wire Line
 	4300 2900 4500 2900
 Wire Wire Line
-	4500 3000 4300 3000
-Wire Wire Line
-	4300 3200 4500 3200
-Wire Wire Line
 	4500 3300 4300 3300
 Wire Wire Line
-	4300 3400 4500 3400
-Wire Wire Line
 	4500 3500 4300 3500
 Wire Wire Line
-	4300 3600 4500 3600
-Wire Wire Line
 	4500 3700 4300 3700
 Wire Wire Line
-	4300 3800 4500 3800
-Wire Wire Line
 	4500 3900 4300 3900
 Wire Wire Line
@@
 Wire Wire Line
 	4300 4200 4500 4200
-Wire Wire Line
-	4500 4300 4300 4300
-Wire Wire Line
-	4300 4400 4500 4400
 Text GLabel 4500 4600 2    50   Input ~ 0
 P1.00
@@
 	4500 4700 4300 4700
 Wire Wire Line
-	4300 4800 4500 4800
-Wire Wire Line
-	4500 4900 4300 4900
-Wire Wire Line
 	4500 5000 4300 5000
 Wire Wire Line
 	4300 5100 4500 5100
 Wire Wire Line
-	4500 5200 4300 5200
-Wire Wire Line
-	4300 5300 4500 5300
-Wire Wire Line
 	4500 5400 4300 5400
 Wire Wire Line
 	4300 5500 4500 5500
 Wire Wire Line
-	4500 5600 4300 5600
-Wire Wire Line
-	4300 5700 4500 5700
-Wire Wire Line
 	4500 5800 4300 5800
 Wire Wire Line
 	4300 5900 4500 5900
-Wire Wire Line
-	4500 6000 4300 6000
-Wire Wire Line
-	4300 6100 4500 6100
 Text GLabel 4500 4400 2    50   Input ~ 0
 P0.31
@@
 Wire Wire Line
 	8550 3550 8550 3400
+$Comp
+L nrf52840-qiaa:nRF52840-QIAA U?
+U 1 1 5C7CF4B7
+P 3200 3700
+F 0 "U?" H 3200 6387 60  0000 C CNN
+F 1 "nRF52840-QIAA" H 3200 6281 60  0000 C CNN
+F 2 "" H 3300 3600 60  0001 C CNN
+F 3 "" H 3300 3600 60  0001 C CNN
+	1    3200 3700
+	-1   0    0    -1
+$EndComp
+Wire Wire Line
+	4300 1400 5400 1400
+Wire Wire Line
+	4300 1300 5400 1300
+Wire Wire Line
+	4300 1500 4500 1500
+Wire Wire Line
+	4300 1600 4500 1600
+Wire Wire Line
+	4300 1700 4500 1700
+Wire Wire Line
+	4300 1900 4500 1900
+Wire Wire Line
+	4300 2000 4500 2000
+Wire Wire Line
+	4300 2400 4500 2400
+Wire Wire Line
+	4300 2600 4500 2600
+Wire Wire Line
+	4300 2800 4500 2800
+Wire Wire Line
+	4300 3000 4500 3000
+Wire Wire Line
+	4300 3200 4500 3200
+Wire Wire Line
+	4300 3400 4500 3400
+Wire Wire Line
+	4300 3600 4500 3600
+Wire Wire Line
+	4300 3800 4500 3800
+Wire Wire Line
+	4300 4300 4500 4300
+Wire Wire Line
+	4300 4400 4500 4400
+Wire Wire Line
+	4300 4800 4500 4800
+Wire Wire Line
+	4300 4900 4500 4900
+Wire Wire Line
+	4300 5200 4500 5200
+Wire Wire Line
+	4300 5300 4500 5300
+Wire Wire Line
+	4300 5600 4500 5600
+Wire Wire Line
+	4300 5700 4500 5700
+Wire Wire Line
+	4300 6000 4500 6000
+Wire Wire Line
+	4300 6100 4500 6100
 $EndSCHEMATC

Commit message: did some cleanup and added power connections
did some cleanup and added power connections
Parts:
- added J?: Conn_ARM_JTAG_SWD_10, Connector_PinHeader_1.27mm:PinHeader_2x05_P1.27mm_Vertical_SMD, symbol Connector:Conn_ARM_JTAG_SWD_10
Connections:
- net labels added: SWDCLK, SWDIO, VSS_BOTT, VSS_b7, usbdata+, usbdata-
- net labels removed: VSS
- wire segments 162 -> 169
Changed lines of the file:
@@
 Text GLabel 1600 5450 3    50   Input ~ 0
 XC1
-Text GLabel 1600 5050 1    50   Input ~ 0
+Text GLabel 1350 4800 1    50   Input ~ 0
 XC2
 Wire Wire Line
@@
 $EndComp
 Wire Wire Line
-	1350 5100 1600 5100
-Wire Wire Line
-	1600 5100 1600 5050
-Wire Wire Line
 	1600 5450 1600 5400
 Wire Wire Line
@@
 $EndComp
 Wire Wire Line
-	1350 5100 1350 4800
-Wire Wire Line
 	1350 4800 1200 4800
 Wire Wire Line
@@
 AR Path="/5C9FDFE4/5CD957DC" Ref="#PWR?"  Part="1"
 AR Path="/5CD957DC" Ref="#PWR?"  Part="1"
-AR Path="/5CD5D522/5CD957DC" Ref="#PWR?"  Part="1"
-F 0 "#PWR?" H 700 5400 50  0001 C CNN
+AR Path="/5CD5D522/5CD957DC" Ref="#PWR0117"  Part="1"
+F 0 "#PWR0117" H 700 5400 50  0001 C CNN
 F 1 "Earth" H 700 5500 50  0001 C CNN
 F 2 "" H 700 5650 50  0001 C CNN
@@
 Ground (VSS_PA)
 Text GLabel 1950 6000 0    50   Input ~ 0
-VSS
+VSS_b7
 Wire Wire Line
 	2100 1400 1950 1400
@@
 	1800 5300 1800 5450
 Wire Wire Line
-	2100 5050 2100 5200
-Wire Wire Line
-	1600 5050 2100 5050
+	2100 5050 2100 5100
 Wire Wire Line
 	1950 5600 2100 5600
@@
 Wire Wire Line
 	4300 6100 4500 6100
+$Comp
+L Connector:Conn_ARM_JTAG_SWD_10 J?
+U 1 1 5C8301A2
+P 7200 4750
+F 0 "J?" H 6760 4796 50  0000 R CNN
+F 1 "Conn_ARM_JTAG_SWD_10" H 6760 4705 50  0000 R CNN
+F 2 "Connector_PinHeader_1.27mm:PinHeader_2x05_P1.27mm_Vertical_SMD" H 7250 4200 50  0001 L TNN
+F 3 "http://infocenter.arm.com/help/topic/com.arm.doc.faqs/attached/13634/cortex_debug_connectors.pdf" V 6850 3500 50  0001 C CNN
+	1    7200 4750
+	1    0    0    -1
+$EndComp
+Text GLabel 1950 4300 0    50   Input ~ 0
+usbdata+
+Text GLabel 1950 4400 0    50   Input ~ 0
+usbdata-
+Text GLabel 1950 6100 0    50   Input ~ 0
+VSS_BOTT
+Text GLabel 1950 4800 0    50   Input ~ 0
+SWDIO
+Text GLabel 1950 4900 0    50   Input ~ 0
+SWDCLK
+Connection ~ 2100 5100
+Wire Wire Line
+	2100 5100 2100 5200
+Wire Wire Line
+	1350 5100 2100 5100
+Wire Wire Line
+	1350 5100 1350 4800
+Wire Wire Line
+	1950 4900 2100 4900
+Wire Wire Line
+	1950 4800 2100 4800
+Wire Wire Line
+	2100 6100 1950 6100
+Wire Wire Line
+	1950 4400 2100 4400
+Wire Wire Line
+	2100 4300 1950 4300
+Text GLabel 7850 4750 2    50   Input ~ 0
+SWDIO
+Text GLabel 7850 4650 2    50   Input ~ 0
+SWDCLK
+Wire Wire Line
+	7850 4650 7700 4650
+Wire Wire Line
+	7850 4750 7700 4750
+Text GLabel 7850 4450 2    50   Input ~ 0
+P0.18
+Wire Wire Line
+	7850 4450 7700 4450
 $EndSCHEMATC

Commit message: worked on power
Connections:
- wire segments 169 -> 172
Changed lines of the file:
@@
 Wire Wire Line
 	7850 4450 7700 4450
+Text GLabel 7200 5500 0    50   Input ~ 0
+VSS_b7
+Wire Wire Line
+	7200 5350 7200 5500
+Text GLabel 7150 3950 0    50   Input ~ 0
+VDD(W1)
+Wire Wire Line
+	7200 4150 7200 3950
+Wire Wire Line
+	7200 3950 7150 3950
 $EndSCHEMATC

Commit message: started pcb
Parts:
- C15, C16: renamed from C?; footprint (none) -> Capacitor_SMD:C_0805_2012Metric_Pad1.15x1.40mm_HandSolder
- J2, J3, J4: renamed from J?; footprint (none) -> Connector_PinHeader_2.54mm:PinHeader_1x02_P2.54mm_Vertical
- J6: renamed from J?; footprint (none) -> Connector_PinHeader_2.54mm:PinHeader_2x20_P2.54mm_Vertical
- P1: renamed from P?; footprint (none) -> Connector_IDC:IDC-Header_2x08_P2.54mm_Vertical
- P2: renamed from P?; footprint (none) -> Connector_IDC:IDC-Header_2x20_P2.54mm_Vertical
- U1: renamed from U?; footprint (none) -> RuuviTag:nRF52840-QIAA
- Y1: renamed from Y?; footprint (none) -> Crystal:Crystal_SMD_2012-2Pin_2.0x1.2mm_HandSoldering
- gave numbers to parts that had none: 1
Connections:
- wire segments 172 -> 175
Changed lines of the file:
@@
 $EndDescr
 $Comp
-L Connector:Raspberry_Pi_2_3 J?
+L Connector:Raspberry_Pi_2_3 J6
 U 1 1 5CD95728
 P 8950 2100
-F 0 "J?" H 8950 3578 50  0000 C CNN
+F 0 "J6" H 8950 3578 50  0000 C CNN
 F 1 "Raspberry_Pi_2_3" H 8950 3487 50  0000 C CNN
-F 2 "" H 8950 2100 50  0001 C CNN
+F 2 "Connector_PinHeader_2.54mm:PinHeader_2x20_P2.54mm_Vertical" H 8950 2100 50  0001 C CNN
 F 3 "https://www.raspberrypi.org/documentation/hardware/raspberrypi/schematics/rpi_SCH_3bplus_1p0_reduced.pdf" H 8950 2100 50  0001 C CNN
 	1    8950 2100
@@
 $EndComp
 $Comp
-L Connector:Conn_01x02_Male J?
+L Connector:Conn_01x02_Male J3
 U 1 1 5CD9572F
 P 5950 900
-F 0 "J?" H 6056 1078 50  0000 C CNN
+F 0 "J3" H 6056 1078 50  0000 C CNN
 F 1 "52840 tx pri rx" H 6056 987 50  0000 C CNN
-F 2 "" H 5950 900 50  0001 C CNN
+F 2 "Connector_PinHeader_2.54mm:PinHeader_1x02_P2.54mm_Vertical" H 5950 900 50  0001 C CNN
 F 3 "~" H 5950 900 50  0001 C CNN
 	1    5950 900
@@
 $EndComp
 $Comp
-L Connector:Conn_01x02_Male J?
+L Connector:Conn_01x02_Male J4
 U 1 1 5CD95736
 P 6400 900
-F 0 "J?" H 6506 1078 50  0000 C CNN
+F 0 "J4" H 6506 1078 50  0000 C CNN
 F 1 "52840 rx rpi tx" H 6506 987 50  0000 C CNN
-F 2 "" H 6400 900 50  0001 C CNN
+F 2 "Connector_PinHeader_2.54mm:PinHeader_1x02_P2.54mm_Vertical" H 6400 900 50  0001 C CNN
 F 3 "~" H 6400 900 50  0001 C CNN
 	1    6400 900
@@
 	6300 1100 6300 1400
 $Comp
-L Connector_Generic:Conn_02x20_Odd_Even P?
+L Connector_Generic:Conn_02x20_Odd_Even P2
 U 1 1 5CD95746
 P 10350 5300
-F 0 "P?" H 10400 6417 50  0000 C CNN
+F 0 "P2" H 10400 6417 50  0000 C CNN
 F 1 "Conn_02x20_Odd_Even" H 10400 6326 50  0000 C CNN
-F 2 "" H 10350 5300 50  0001 C CNN
+F 2 "Connector_IDC:IDC-Header_2x20_P2.54mm_Vertical" H 10350 5300 50  0001 C CNN
 F 3 "~" H 10350 5300 50  0001 C CNN
 	1    10350 5300
@@
       _n____n__\n     /         \---||--<\n    /___________\\n    _|____|____|_\n    _|____|____|_\n     |    |    |\n    --------------\n    | || || || ||\\n    | || || || || \++++++++------<\n    ===============\n    |   |  |  |   |\n   (| O | O| O| O |)\n   |   |   |   |   |\n  (| O | O | O | O |)\n   |   |   |   |    |\n (| O |  O | O  | O |)\n  |   |    |    |    |\n (| O |  O |  O |  O |)\n ======================
 $Comp
-L Connector_Generic:Conn_02x08_Odd_Even P?
+L Connector_Generic:Conn_02x08_Odd_Even P1
 U 1 1 5CD95789
 P 8800 5900
-F 0 "P?" H 8850 6417 50  0000 C CNN
+F 0 "P1" H 8850 6417 50  0000 C CNN
 F 1 "Conn_02x08_Odd_Even" H 8850 6326 50  0000 C CNN
-F 2 "" H 8800 5900 50  0001 C CNN
+F 2 "Connector_IDC:IDC-Header_2x08_P2.54mm_Vertical" H 8800 5900 50  0001 C CNN
 F 3 "~" H 8800 5900 50  0001 C CNN
 	1    8800 5900
@@
 	1800 5450 1600 5450
 $Comp
-L Device:Crystal Y?
+L Device:Crystal Y1
 U 1 1 5CD957BB
 P 900 5250
-F 0 "Y?" V 946 5119 50  0000 R CNN
+F 0 "Y1" V 946 5119 50  0000 R CNN
 F 1 "32mhzCrystal" V 855 5119 50  0000 R CNN
-F 2 "" H 900 5250 50  0001 C CNN
+F 2 "Crystal:Crystal_SMD_2012-2Pin_2.0x1.2mm_HandSoldering" H 900 5250 50  0001 C CNN
 F 3 "~" H 900 5250 50  0001 C CNN
 	1    900  5250
@@
 	1600 5400 1350 5400
 $Comp
-L Device:C_Small C?
+L Device:C_Small C16
 U 1 1 5CD957C6
 P 1100 5600
-F 0 "C?" V 871 5600 50  0000 C CNN
+F 0 "C16" V 871 5600 50  0000 C CNN
 F 1 "12pf" V 962 5600 50  0000 C CNN
-F 2 "" H 1100 5600 50  0001 C CNN
+F 2 "Capacitor_SMD:C_0805_2012Metric_Pad1.15x1.40mm_HandSolder" H 1100 5600 50  0001 C CNN
 F 3 "~" H 1100 5600 50  0001 C CNN
 	1    1100 5600
@@
 $EndComp
 $Comp
-L Device:C_Small C?
+L Device:C_Small C15
 U 1 1 5CD957CD
 P 1100 4800
-F 0 "C?" V 871 4800 50  0000 C CNN
+F 0 "C15" V 871 4800 50  0000 C CNN
 F 1 "12pf" V 962 4800 50  0000 C CNN
-F 2 "" H 1100 4800 50  0001 C CNN
+F 2 "Capacitor_SMD:C_0805_2012Metric_Pad1.15x1.40mm_HandSolder" H 1100 4800 50  0001 C CNN
 F 3 "~" H 1100 4800 50  0001 C CNN
 	1    1100 4800
@@
 VSS_b7
 Wire Wire Line
-	2100 1400 1950 1400
-Wire Wire Line
-	2100 1900 1950 1900
-Wire Wire Line
-	2100 2000 1950 2000
-Wire Wire Line
-	2100 2400 1950 2400
-Wire Wire Line
-	1950 2600 2100 2600
-Wire Wire Line
-	2100 2800 1950 2800
-Wire Wire Line
-	2100 3000 1950 3000
-Wire Wire Line
-	1950 3200 2100 3200
-Wire Wire Line
-	2100 3400 1950 3400
-Wire Wire Line
-	1950 3600 2100 3600
-Wire Wire Line
-	2100 3800 1950 3800
-Wire Wire Line
 	2100 4500 1850 4500
 Wire Wire Line
@@
 	1950 5700 1950 5850
 Wire Wire Line
-	1950 6000 2100 6000
-$Comp
-L Connector:Conn_01x02_Male J?
+	1950 6000 2050 6000
+$Comp
+L Connector:Conn_01x02_Male J2
 U 1 1 5CD95808
 P 5600 2300
-F 0 "J?" H 5572 2180 50  0000 R CNN
+F 0 "J2" H 5572 2180 50  0000 R CNN
 F 1 "nfc " H 5572 2271 50  0000 R CNN
-F 2 "" H 5600 2300 50  0001 C CNN
+F 2 "Connector_PinHeader_2.54mm:PinHeader_1x02_P2.54mm_Vertical" H 5600 2300 50  0001 C CNN
 F 3 "~" H 5600 2300 50  0001 C CNN
 	1    5600 2300
@@
 	4500 3300 4300 3300
 Wire Wire Line
-	4500 3500 4300 3500
-Wire Wire Line
 	4500 3700 4300 3700
 Wire Wire Line
@@
 Text GLabel 1950 1300 0    50   Input ~ 0
 VDD(A22)
-Wire Wire Line
-	2100 1300 1950 1300
-Wire Wire Line
-	2100 1500 1950 1500
-Wire Wire Line
-	2100 1600 1950 1600
-Wire Wire Line
-	2100 1700 1950 1700
 Text GLabel 8100 750  0    50   Input ~ 0
 rpi(5v)(pin2)
@@
 	8550 3550 8550 3400
 $Comp
-L nrf52840-qiaa:nRF52840-QIAA U?
+L nrf52840-qiaa:nRF52840-QIAA U1
 U 1 1 5C7CF4B7
 P 3200 3700
-F 0 "U?" H 3200 6387 60  0000 C CNN
+F 0 "U1" H 3200 6387 60  0000 C CNN
 F 1 "nRF52840-QIAA" H 3200 6281 60  0000 C CNN
-F 2 "" H 3300 3600 60  0001 C CNN
+F 2 "RuuviTag:nRF52840-QIAA" H 3300 3600 60  0001 C CNN
 F 3 "" H 3300 3600 60  0001 C CNN
 	1    3200 3700
@@
 	4300 6100 4500 6100
 $Comp
-L Connector:Conn_ARM_JTAG_SWD_10 J?
+L Connector:Conn_ARM_JTAG_SWD_10 J5
 U 1 1 5C8301A2
 P 7200 4750
-F 0 "J?" H 6760 4796 50  0000 R CNN
+F 0 "J5" H 6760 4796 50  0000 R CNN
 F 1 "Conn_ARM_JTAG_SWD_10" H 6760 4705 50  0000 R CNN
 F 2 "Connector_PinHeader_1.27mm:PinHeader_2x05_P1.27mm_Vertical_SMD" H 7250 4200 50  0001 L TNN
@@
 	1950 4800 2100 4800
 Wire Wire Line
-	2100 6100 1950 6100
+	2100 6100 2050 6100
 Wire Wire Line
 	1950 4400 2100 4400
@@
 Wire Wire Line
 	7200 3950 7150 3950
+Wire Wire Line
+	2050 6100 2050 6000
+Connection ~ 2050 6100
+Wire Wire Line
+	2050 6100 1950 6100
+Connection ~ 2050 6000
+Wire Wire Line
+	2050 6000 2100 6000
+Wire Wire Line
+	2100 1300 1950 1300
+Wire Wire Line
+	1950 1400 2100 1400
+Wire Wire Line
+	2100 1500 1950 1500
+Wire Wire Line
+	1950 1600 2100 1600
+Wire Wire Line
+	2100 1700 1950 1700
+Wire Wire Line
+	1950 1900 2100 1900
+Wire Wire Line
+	2100 2000 1950 2000
+Wire Wire Line
+	2100 2400 1950 2400
+Wire Wire Line
+	2100 2600 1950 2600
+Wire Wire Line
+	2100 2800 1950 2800
+Wire Wire Line
+	2100 3000 1950 3000
+Wire Wire Line
+	1950 3200 2100 3200
+Wire Wire Line
+	2100 3400 1950 3400
+Wire Wire Line
+	1950 3600 2100 3600
+Wire Wire Line
+	2100 3800 1950 3800
+Wire Wire Line
+	4300 3500 4500 3500
 $EndSCHEMATC

Commit message: added reference files
Connections:
- wire segments 175 -> 178
Changed lines of the file:
@@
 	1950 3200 2100 3200
 Wire Wire Line
-	2100 3400 1950 3400
+	2100 3400 2000 3400
 Wire Wire Line
-	1950 3600 2100 3600
+	1950 3600 2000 3600
 Wire Wire Line
 	2100 3800 1950 3800
 Wire Wire Line
 	4300 3500 4500 3500
+Text GLabel 3350 7000 0    50   Input ~ 0
+1.3vsup_decup(dec4)
+Wire Wire Line
+	2000 3600 2000 3400
+Connection ~ 2000 3600
+Wire Wire Line
+	2000 3600 2100 3600
+Connection ~ 2000 3400
+Wire Wire Line
+	2000 3400 1950 3400
 $EndSCHEMATC
