File: hat/nrf52840-and-connectors.sch (KiCad schematic (older format))
At the start: 11 parts, among them J2 nfc, J3 52840 tx pri rx, J4 52840 rx rpi tx, J5 Conn_ARM_JTAG_SWD_10, J6 Raspberry_Pi_2_3, P1 Conn_02x08_Odd_Even, P2 Conn_02x20_Odd_Even, U1 nRF52840-QIAA, Y1 32mhzCrystal

Commit message: added basic varient
Parts:
- removed C15, C16: 12pf, Capacitor_SMD:C_0805_2012Metric_Pad1.15x1.40mm_HandSolder, symbol Device:C_Small
- removed P1: Conn_02x08_Odd_Even, Connector_IDC:IDC-Header_2x08_P2.54mm_Vertical, symbol Connector_Generic:Conn_02x08_Odd_Even
- removed P2: Conn_02x20_Odd_Even, Connector_IDC:IDC-Header_2x20_P2.54mm_Vertical, symbol Connector_Generic:Conn_02x20_Odd_Even
- removed U1: nRF52840-QIAA, RuuviTag:nRF52840-QIAA, symbol nrf52840-qiaa:nRF52840-QIAA
- removed Y1: 32mhzCrystal, Crystal:Crystal_SMD_2012-2Pin_2.0x1.2mm_HandSoldering, symbol Device:Crystal
- added U1: nrf52840, nordic:nrf52840, symbol nordic:nrf52840
- renumbered J6 to J5, J5 to J6
Connections:
- net labels added: VDD(AD14)
- net labels removed: Earth, VDD(A14)
- wire segments 178 -> 158
Other:
- note added: "This is for dev version\naka prototypers delight"

Commit message: optimized layout
Parts:
- J6: symbol Connector:Conn_ARM_JTAG_SWD_10 -> hat-rescue:Conn_ARM_JTAG_SWD_10-Connector
Changed lines of the file:
@@
 EESchema Schematic File Version 4
 LIBS:hat-cache
-EELAYER 26 0
+EELAYER 29 0
 EELAYER END
 $Descr A4 11693 8268
@@
 	2300 2800 2100 2800
 $Comp
-L Connector:Conn_ARM_JTAG_SWD_10 J6
+L hat-rescue:Conn_ARM_JTAG_SWD_10-Connector J6
 U 1 1 5C8301A2
 P 10200 4450
+AR Path="/5C8301A2" Ref="J6"  Part="1"
+AR Path="/5CD5D522/5C8301A2" Ref="J6"  Part="1"
 F 0 "J6" H 9760 4496 50  0000 R CNN
 F 1 "Conn_ARM_JTAG_SWD_10" H 9760 4405 50  0000 R CNN
