File: hat/basic-hat.kicad_pcb (KiCad board)
At the start: 4 copper layers, 45 parts, among them IC1 LM2676S-5.0, IC2 DMMT5401-7-F, J1 Conn_Coaxial, J2 nfc, J3 52840 tx pri rx, J4 52840 rx rpi tx, J5 Raspberry_Pi_2_3, J6 Conn_ARM_JTAG_SWD_10, J7 Screw_Terminal_01x02, J8 Screw_Terminal_01x01, Q1 DMG2305UX-7, U1 nrf52840, Y1 32mhzCrystal

Commit message: added basic varient
Parts:
- moved J4 10.2 mm to (89.7, 30.0)
- moved J3 10.2 mm to (93.4, 30.0)
- moved J6 10.2 mm to (82.0, 31.8)
- moved U1 5.64 mm to (76.5, 49.3), turned to 0 degrees
- moved J7 4.83 mm to (47.2, 32.0), turned to 270 degrees
- moved C22 0.34 mm to (50.3, 52.8), turned to 0 degrees
Routing:
- net Ground (VSS_PA): track 189.5 -> 0.00 mm, vias 4 -> 0
- net VDDH: track 78.2 -> 0.00 mm
- net +12V: track 48.0 -> 0.00 mm
- net Net-(C22-Pad1): track 36.0 -> 0.00 mm, vias 2 -> 0
- net Net-(J3-Pad1): track 30.0 -> 0.00 mm
- net Net-(J4-Pad1): track 28.3 -> 0.00 mm
- net VDD(A22): track 23.5 -> 0.00 mm, vias 2 -> 0
- net Net-(IC1-Pad7): track 22.4 -> 0.00 mm, vias 2 -> 0
- net Net-(C21-Pad1): track 21.1 -> 0.00 mm, vias 2 -> 0
- net Net-(ANT1-Pad1): track 17.3 -> 0.00 mm
- net DCC: track 12.6 -> 0.00 mm, vias 2 -> 0
- net ant: track 12.6 -> 0.00 mm
- net 1.3vsup_decup(dec4): track 12.0 -> 0.00 mm, vias 2 -> 0
- net Net-(IC2-Pad1): track 9.28 -> 0.00 mm
- net Net-(C11-Pad1): track 6.75 -> 0.00 mm
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
Commit message: vega
Parts:
- turned U1 to 180 degrees
Routing:
- net Ground (VSS_PA): track 0.00 -> 235.6 mm
- net VDDH: track 0.00 -> 75.7 mm, vias 0 -> 3
- net +12V: track 0.00 -> 47.4 mm, vias 0 -> 2
- net Net-(J3-Pad1): track 0.00 -> 39.2 mm
- net Net-(C22-Pad1): track 0.00 -> 37.6 mm, vias 0 -> 2
- net Net-(J4-Pad1): track 0.00 -> 37.3 mm
- net Net-(IC1-Pad7): track 0.00 -> 23.4 mm, vias 0 -> 2
- net ant: track 0.00 -> 18.3 mm
- net Net-(C21-Pad1): track 0.00 -> 18.2 mm
- net Net-(ANT1-Pad1): track 0.00 -> 16.9 mm
- net VDD(A22): track 0.00 -> 11.4 mm
- net Net-(IC2-Pad1): track 0.00 -> 9.28 mm
- net Net-(IC2-Pad4): track 0.00 -> 7.59 mm
- net Net-(C11-Pad1): track 0.00 -> 7.27 mm
- net 1.3vsup_decup(dec4): track 0.00 -> 5.45 mm
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Other:
- board outline added: 65 x 56.5 mm

Commit message: basicly done basic version
NOT COMPLEATED YET but close
Parts:
- moved J2 2.55 mm to (87.1, 74.7), turned to 270 degrees
Routing:
- net VDD(A22): track 11.4 -> 91.4 mm, vias 0 -> 9
- net 1.3vsup_decup(dec4): track 5.45 -> 50.3 mm, vias 0 -> 3
- net P0.09: track 0.00 -> 40.6 mm, vias 0 -> 1
- net P0.10: track 0.00 -> 38.4 mm, vias 0 -> 1
- net 1.3vsup_decup(flash)(dec5): track 0.00 -> 35.6 mm, vias 0 -> 2
- net SWDCLK: track 0.00 -> 34.6 mm, vias 0 -> 2
- net psu_decup(dec3): track 0.00 -> 31.9 mm, vias 0 -> 2
- net P0.01: track 0.00 -> 30.8 mm
- net SWDIO: track 0.00 -> 30.6 mm
- net XC1: track 0.00 -> 29.2 mm, vias 0 -> 2
- net p0.00: track 0.00 -> 27.9 mm
- net DCC: track 0.00 -> 26.3 mm, vias 0 -> 2
- net DCCH: track 0.00 -> 25.4 mm, vias 0 -> 2
- net 1.1vsup_decup(dec1): track 0.00 -> 24.7 mm, vias 0 -> 2
- net VDDH: track 75.7 -> 99.7 mm, vias 3 -> 5
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Other:
- net class Default: clearance 0.2 -> 0.19
- rule trace_clearance: 0.2 -> 0.19
- rule via_min_drill: 0.35 -> 0.1
