File: hat/dafault-config.sch (KiCad schematic (older format))
At the start: 20 parts

Commit message: started pcb
Parts:
- ANT1: renamed from ANT?; footprint CONUFL001-SMD -> SamacSys_Parts:CONUFL001-SMD
- C1, C10, C11, C12, C13, C14, C2, C3, C4, C5, C6, C7, C8, C9: renamed from C?; footprint (none) -> Capacitor_SMD:C_0805_2012Metric_Pad1.15x1.40mm_HandSolder
- J1: renamed from J?; footprint (none) -> Connector_Coaxial:SMA_Amphenol_132134-16_Vertical
- L1, L2, L3, L4: renamed from L?; footprint (none) -> Inductor_SMD:L_0805_2012Metric_Pad1.15x1.40mm_HandSolder
Changed lines of the file:
@@
 P 7000 850
 AR Path="/5CC155B9" Ref="C?"  Part="1"
-AR Path="/5C9FDFE4/5CC155B9" Ref="C?"  Part="1"
-F 0 "C?" V 6771 850 50  0000 C CNN
+AR Path="/5C9FDFE4/5CC155B9" Ref="C1"  Part="1"
+F 0 "C1" V 6771 850 50  0000 C CNN
 F 1 "100nF" V 6862 850 50  0000 C CNN
-F 2 "" H 7000 850 50  0001 C CNN
+F 2 "Capacitor_SMD:C_0805_2012Metric_Pad1.15x1.40mm_HandSolder" H 7000 850 50  0001 C CNN
 F 3 "~" H 7000 850 50  0001 C CNN
 	1    7000 850
@@
 P 7000 1400
 AR Path="/5CC155E6" Ref="C?"  Part="1"
-AR Path="/5C9FDFE4/5CC155E6" Ref="C?"  Part="1"
-F 0 "C?" V 6771 1400 50  0000 C CNN
+AR Path="/5C9FDFE4/5CC155E6" Ref="C2"  Part="1"
+F 0 "C2" V 6771 1400 50  0000 C CNN
 F 1 "1.0uF" V 6862 1400 50  0000 C CNN
-F 2 "" H 7000 1400 50  0001 C CNN
+F 2 "Capacitor_SMD:C_0805_2012Metric_Pad1.15x1.40mm_HandSolder" H 7000 1400 50  0001 C CNN
 F 3 "~" H 7000 1400 50  0001 C CNN
 	1    7000 1400
@@
 P 7000 3150
 AR Path="/5CC15601" Ref="C?"  Part="1"
-AR Path="/5C9FDFE4/5CC15601" Ref="C?"  Part="1"
-F 0 "C?" V 6771 3150 50  0000 C CNN
+AR Path="/5C9FDFE4/5CC15601" Ref="C7"  Part="1"
+F 0 "C7" V 6771 3150 50  0000 C CNN
 F 1 "407uF" V 6862 3150 50  0000 C CNN
-F 2 "" H 7000 3150 50  0001 C CNN
+F 2 "Capacitor_SMD:C_0805_2012Metric_Pad1.15x1.40mm_HandSolder" H 7000 3150 50  0001 C CNN
 F 3 "~" H 7000 3150 50  0001 C CNN
 	1    7000 3150
@@
 P 9300 1050
 AR Path="/5CC1560F" Ref="C?"  Part="1"
-AR Path="/5C9FDFE4/5CC1560F" Ref="C?"  Part="1"
-F 0 "C?" H 9208 1004 50  0000 R CNN
+AR Path="/5C9FDFE4/5CC1560F" Ref="C12"  Part="1"
+F 0 "C12" H 9208 1004 50  0000 R CNN
 F 1 "0.5pF" H 9208 1095 50  0000 R CNN
-F 2 "" H 9300 1050 50  0001 C CNN
+F 2 "Capacitor_SMD:C_0805_2012Metric_Pad1.15x1.40mm_HandSolder" H 9300 1050 50  0001 C CNN
 F 3 "~" H 9300 1050 50  0001 C CNN
 	1    9300 1050
@@
 P 8700 1050
 AR Path="/5CC1562A" Ref="C?"  Part="1"
-AR Path="/5C9FDFE4/5CC1562A" Ref="C?"  Part="1"
-F 0 "C?" H 8792 1096 50  0000 L CNN
+AR Path="/5C9FDFE4/5CC1562A" Ref="C11"  Part="1"
+F 0 "C11" H 8792 1096 50  0000 L CNN
 F 1 "0.8pF" H 8792 1005 50  0000 L CNN
-F 2 "" H 8700 1050 50  0001 C CNN
+F 2 "Capacitor_SMD:C_0805_2012Metric_Pad1.15x1.40mm_HandSolder" H 8700 1050 50  0001 C CNN
 F 3 "~" H 8700 1050 50  0001 C CNN
 	1    8700 1050
@@
 P 10050 3000
 AR Path="/5CC15663" Ref="C?"  Part="1"
-AR Path="/5C9FDFE4/5CC15663" Ref="C?"  Part="1"
-F 0 "C?" V 9821 3000 50  0000 C CNN
+AR Path="/5C9FDFE4/5CC15663" Ref="C14"  Part="1"
+F 0 "C14" V 9821 3000 50  0000 C CNN
 F 1 "1.0uf" V 9912 3000 50  0000 C CNN
-F 2 "" H 10050 3000 50  0001 C CNN
+F 2 "Capacitor_SMD:C_0805_2012Metric_Pad1.15x1.40mm_HandSolder" H 10050 3000 50  0001 C CNN
 F 3 "~" H 10050 3000 50  0001 C CNN
 	1    10050 3000
@@
 P 7000 2850
 AR Path="/5CC15676" Ref="C?"  Part="1"
-AR Path="/5C9FDFE4/5CC15676" Ref="C?"  Part="1"
-F 0 "C?" V 6771 2850 50  0000 C CNN
+AR Path="/5C9FDFE4/5CC15676" Ref="C6"  Part="1"
+F 0 "C6" V 6771 2850 50  0000 C CNN
 F 1 "4.7uf" V 6862 2850 50  0000 C CNN
-F 2 "" H 7000 2850 50  0001 C CNN
+F 2 "Capacitor_SMD:C_0805_2012Metric_Pad1.15x1.40mm_HandSolder" H 7000 2850 50  0001 C CNN
 F 3 "~" H 7000 2850 50  0001 C CNN
 	1    7000 2850
@@
 P 7000 4300
 AR Path="/5CC1568C" Ref="C?"  Part="1"
-AR Path="/5C9FDFE4/5CC1568C" Ref="C?"  Part="1"
-F 0 "C?" V 6771 4300 50  0000 C CNN
+AR Path="/5C9FDFE4/5CC1568C" Ref="C10"  Part="1"
+F 0 "C10" V 6771 4300 50  0000 C CNN
 F 1 "nc" V 6862 4300 50  0000 C CNN
-F 2 "" H 7000 4300 50  0001 C CNN
+F 2 "Capacitor_SMD:C_0805_2012Metric_Pad1.15x1.40mm_HandSolder" H 7000 4300 50  0001 C CNN
 F 3 "~" H 7000 4300 50  0001 C CNN
 	1    7000 4300
@@
 P 7000 3950
 AR Path="/5CC156A1" Ref="C?"  Part="1"
-AR Path="/5C9FDFE4/5CC156A1" Ref="C?"  Part="1"
-F 0 "C?" V 6771 3950 50  0000 C CNN
+AR Path="/5C9FDFE4/5CC156A1" Ref="C9"  Part="1"
+F 0 "C9" V 6771 3950 50  0000 C CNN
 F 1 "nc" V 6862 3950 50  0000 C CNN
-F 2 "" H 7000 3950 50  0001 C CNN
+F 2 "Capacitor_SMD:C_0805_2012Metric_Pad1.15x1.40mm_HandSolder" H 7000 3950 50  0001 C CNN
 F 3 "~" H 7000 3950 50  0001 C CNN
 	1    7000 3950
@@
 P 7000 3500
 AR Path="/5CC156D1" Ref="C?"  Part="1"
-AR Path="/5C9FDFE4/5CC156D1" Ref="C?"  Part="1"
-F 0 "C?" V 6771 3500 50  0000 C CNN
+AR Path="/5C9FDFE4/5CC156D1" Ref="C8"  Part="1"
+F 0 "C8" V 6771 3500 50  0000 C CNN
 F 1 "4.7uf" V 6862 3500 50  0000 C CNN
-F 2 "" H 7000 3500 50  0001 C CNN
+F 2 "Capacitor_SMD:C_0805_2012Metric_Pad1.15x1.40mm_HandSolder" H 7000 3500 50  0001 C CNN
 F 3 "~" H 7000 3500 50  0001 C CNN
 	1    7000 3500
@@
 P 7000 1800
 AR Path="/5CC5F901" Ref="C?"  Part="1"
-AR Path="/5C9FDFE4/5CC5F901" Ref="C?"  Part="1"
-F 0 "C?" V 6771 1800 50  0000 C CNN
+AR Path="/5C9FDFE4/5CC5F901" Ref="C3"  Part="1"
+F 0 "C3" V 6771 1800 50  0000 C CNN
 F 1 "1.0uF" V 6862 1800 50  0000 C CNN
-F 2 "" H 7000 1800 50  0001 C CNN
+F 2 "Capacitor_SMD:C_0805_2012Metric_Pad1.15x1.40mm_HandSolder" H 7000 1800 50  0001 C CNN
 F 3 "~" H 7000 1800 50  0001 C CNN
 	1    7000 1800
@@
 P 7000 2150
 AR Path="/5CC5F925" Ref="C?"  Part="1"
-AR Path="/5C9FDFE4/5CC5F925" Ref="C?"  Part="1"
-F 0 "C?" V 6771 2150 50  0000 C CNN
+AR Path="/5C9FDFE4/5CC5F925" Ref="C4"  Part="1"
+F 0 "C4" V 6771 2150 50  0000 C CNN
 F 1 "1.0uF" V 6862 2150 50  0000 C CNN
-F 2 "" H 7000 2150 50  0001 C CNN
+F 2 "Capacitor_SMD:C_0805_2012Metric_Pad1.15x1.40mm_HandSolder" H 7000 2150 50  0001 C CNN
 F 3 "~" H 7000 2150 50  0001 C CNN
 	1    7000 2150
@@
 P 9400 3850
 AR Path="/5CC5F94E" Ref="C?"  Part="1"
-AR Path="/5C9FDFE4/5CC5F94E" Ref="C?"  Part="1"
-F 0 "C?" V 9171 3850 50  0000 C CNN
+AR Path="/5C9FDFE4/5CC5F94E" Ref="C13"  Part="1"
+F 0 "C13" V 9171 3850 50  0000 C CNN
 F 1 "1.0uF" V 9262 3850 50  0000 C CNN
-F 2 "" H 9400 3850 50  0001 C CNN
+F 2 "Capacitor_SMD:C_0805_2012Metric_Pad1.15x1.40mm_HandSolder" H 9400 3850 50  0001 C CNN
 F 3 "~" H 9400 3850 50  0001 C CNN
 	1    9400 3850
@@
 	9300 1150 9300 1400
 $Comp
-L Device:L L?
+L Device:L L1
 U 1 1 5CC7FBEF
 P 9000 800
-F 0 "L?" V 9190 800 50  0000 C CNN
+F 0 "L1" V 9190 800 50  0000 C CNN
 F 1 "3.3nH" V 9099 800 50  0000 C CNN
-F 2 "" H 9000 800 50  0001 C CNN
+F 2 "Inductor_SMD:L_0805_2012Metric_Pad1.15x1.40mm_HandSolder" H 9000 800 50  0001 C CNN
 F 3 "~" H 9000 800 50  0001 C CNN
 	1    9000 800
@@
 VSS_b7
 $Comp
-L Device:L L?
+L Device:L L3
 U 1 1 5CC9371F
 P 9200 3000
-F 0 "L?" V 9390 3000 50  0000 C CNN
+F 0 "L3" V 9390 3000 50  0000 C CNN
 F 1 "10uH" V 9299 3000 50  0000 C CNN
-F 2 "" H 9200 3000 50  0001 C CNN
+F 2 "Inductor_SMD:L_0805_2012Metric_Pad1.15x1.40mm_HandSolder" H 9200 3000 50  0001 C CNN
 F 3 "~" H 9200 3000 50  0001 C CNN
 	1    9200 3000
@@
 $EndComp
 $Comp
-L Device:L L?
+L Device:L L4
 U 1 1 5CC93DA2
 P 9650 3000
-F 0 "L?" V 9840 3000 50  0000 C CNN
+F 0 "L4" V 9840 3000 50  0000 C CNN
 F 1 "15nH" V 9749 3000 50  0000 C CNN
-F 2 "" H 9650 3000 50  0001 C CNN
+F 2 "Inductor_SMD:L_0805_2012Metric_Pad1.15x1.40mm_HandSolder" H 9650 3000 50  0001 C CNN
 F 3 "~" H 9650 3000 50  0001 C CNN
 	1    9650 3000
@@
 P 7000 2500
 AR Path="/5CC9F77D" Ref="C?"  Part="1"
-AR Path="/5C9FDFE4/5CC9F77D" Ref="C?"  Part="1"
-F 0 "C?" V 6771 2500 50  0000 C CNN
+AR Path="/5C9FDFE4/5CC9F77D" Ref="C5"  Part="1"
+F 0 "C5" V 6771 2500 50  0000 C CNN
 F 1 "1.0uF" V 6862 2500 50  0000 C CNN
-F 2 "" H 7000 2500 50  0001 C CNN
+F 2 "Capacitor_SMD:C_0805_2012Metric_Pad1.15x1.40mm_HandSolder" H 7000 2500 50  0001 C CNN
 F 3 "~" H 7000 2500 50  0001 C CNN
 	1    7000 2500
@@
 	9600 3850 9700 3850
 $Comp
-L Device:L L?
+L Device:L L2
 U 1 1 5CCA8CFC
 P 9100 3650
-F 0 "L?" V 9290 3650 50  0000 C CNN
+F 0 "L2" V 9290 3650 50  0000 C CNN
 F 1 "10uH" V 9199 3650 50  0000 C CNN
-F 2 "" H 9100 3650 50  0001 C CNN
+F 2 "Inductor_SMD:L_0805_2012Metric_Pad1.15x1.40mm_HandSolder" H 9100 3650 50  0001 C CNN
 F 3 "~" H 9100 3650 50  0001 C CNN
 	1    9100 3650
@@
 	6800 2850 6700 2850
 $Comp
-L Connector:Conn_Coaxial J?
+L Connector:Conn_Coaxial J1
 U 1 1 5C8668E2
 P 10850 800
-F 0 "J?" H 10949 776 50  0000 L CNN
+F 0 "J1" H 10949 776 50  0000 L CNN
 F 1 "Conn_Coaxial" H 10949 685 50  0000 L CNN
-F 2 "" H 10850 800 50  0001 C CNN
+F 2 "Connector_Coaxial:SMA_Amphenol_132134-16_Vertical" H 10850 800 50  0001 C CNN
 F 3 " ~" H 10850 800 50  0001 C CNN
 	1    10850 800
@@
 $EndComp
 $Comp
-L power:Earth #PWR?
+L power:Earth #PWR0103
 U 1 1 5C8694A0
 P 11100 1800
-F 0 "#PWR?" H 11100 1550 50  0001 C CNN
+F 0 "#PWR0103" H 11100 1550 50  0001 C CNN
 F 1 "Earth" H 11100 1650 50  0001 C CNN
 F 2 "" H 11100 1800 50  0001 C CNN
@@
 	11100 1750 11100 1800
 $Comp
-L SamacSys_Parts:CONUFL001-SMD ANT?
+L SamacSys_Parts:CONUFL001-SMD ANT1
 U 1 1 5C885D44
 P 10250 1100
-F 0 "ANT?" H 10850 1365 50  0000 C CNN
+F 0 "ANT1" H 10850 1365 50  0000 C CNN
 F 1 "CONUFL001-SMD" H 10850 1274 50  0000 C CNN
-F 2 "CONUFL001-SMD" H 11300 1200 50  0001 L CNN
+F 2 "SamacSys_Parts:CONUFL001-SMD" H 11300 1200 50  0001 L CNN
 F 3 "https://componentsearchengine.com/Datasheets/1/CONUFL001-SMD.pdf" H 11300 1100 50  0001 L CNN
 F 4 "RF Connectors / Coaxial Connectors U.FL Straight Surface Mount Jack" H 11300 1000 50  0001 L CNN "Description"

Commit message: added reference files
Parts:
- removed C11: 0.8pF, Capacitor_SMD:C_0805_2012Metric_Pad1.15x1.40mm_HandSolder, symbol Device:C_Small
- removed C12: 0.5pF, Capacitor_SMD:C_0805_2012Metric_Pad1.15x1.40mm_HandSolder, symbol Device:C_Small
- added C?: 1.0pF, Capacitor_SMD:C_0805_2012Metric_Pad1.15x1.40mm_HandSolder, symbol Device:C_Small
- added L?: 4.7nH, Inductor_SMD:L_0805_2012Metric_Pad1.15x1.40mm_HandSolder, symbol Device:L
- C9: value nc -> 820pf
- L1: value 3.3nH -> 3.9nH
Changed lines of the file:
@@
-$Comp
-L Device:C_Small C?
-U 1 1 5CC1560F
-P 9300 1050
-AR Path="/5CC1560F" Ref="C?"  Part="1"
-AR Path="/5C9FDFE4/5CC1560F" Ref="C12"  Part="1"
-F 0 "C12" H 9208 1004 50  0000 R CNN
-F 1 "0.5pF" H 9208 1095 50  0000 R CNN
-F 2 "Capacitor_SMD:C_0805_2012Metric_Pad1.15x1.40mm_HandSolder" H 9300 1050 50  0001 C CNN
-F 3 "~" H 9300 1050 50  0001 C CNN
-	1    9300 1050
-	-1   0    0    1
-$EndComp
-$Comp
-L Device:C_Small C?
-U 1 1 5CC1562A
-P 8700 1050
-AR Path="/5CC1562A" Ref="C?"  Part="1"
-AR Path="/5C9FDFE4/5CC1562A" Ref="C11"  Part="1"
-F 0 "C11" H 8792 1096 50  0000 L CNN
-F 1 "0.8pF" H 8792 1005 50  0000 L CNN
-F 2 "Capacitor_SMD:C_0805_2012Metric_Pad1.15x1.40mm_HandSolder" H 8700 1050 50  0001 C CNN
-F 3 "~" H 8700 1050 50  0001 C CNN
-	1    8700 1050
-	1    0    0    -1
-$EndComp
 $Comp
 L Device:C_Small C?
@@
 AR Path="/5C9FDFE4/5CC156A1" Ref="C9"  Part="1"
 F 0 "C9" V 6771 3950 50  0000 C CNN
-F 1 "nc" V 6862 3950 50  0000 C CNN
+F 1 "820pf" V 6862 3950 50  0000 C CNN
 F 2 "Capacitor_SMD:C_0805_2012Metric_Pad1.15x1.40mm_HandSolder" H 7000 3950 50  0001 C CNN
 F 3 "~" H 7000 3950 50  0001 C CNN
@@
 $EndComp
 $Comp
-L power:Earth #PWR0107
-U 1 1 5CC15AF4
-P 9300 1400
-F 0 "#PWR0107" H 9300 1150 50  0001 C CNN
-F 1 "Earth" H 9300 1250 50  0001 C CNN
-F 2 "" H 9300 1400 50  0001 C CNN
-F 3 "~" H 9300 1400 50  0001 C CNN
-	1    9300 1400
-	1    0    0    -1
-$EndComp
-$Comp
 L power:Earth #PWR0108
 U 1 1 5CC15B08
@@
 	8500 1300 8700 1300
 Wire Wire Line
-	8700 1300 8700 1150
-Wire Wire Line
 	8700 1300 8700 1400
-Connection ~ 8700 1300
-Wire Wire Line
-	9300 1150 9300 1400
 $Comp
 L Device:L L1
@@
 P 9000 800
 F 0 "L1" V 9190 800 50  0000 C CNN
-F 1 "3.3nH" V 9099 800 50  0000 C CNN
+F 1 "3.9nH" V 9099 800 50  0000 C CNN
 F 2 "Inductor_SMD:L_0805_2012Metric_Pad1.15x1.40mm_HandSolder" H 9000 800 50  0001 C CNN
 F 3 "~" H 9000 800 50  0001 C CNN
@@
 	0    -1   -1   0
 $EndComp
-Wire Wire Line
-	8500 800  8700 800
-Wire Wire Line
-	8700 950  8700 800
-Connection ~ 8700 800
-Wire Wire Line
-	8700 800  8850 800
-Wire Wire Line
-	9150 800  9300 800
-Wire Wire Line
-	9300 800  9300 950
-Connection ~ 9300 800
 Text GLabel 6700 3150 0    50   Input ~ 0
 Vbus
@@
 Connection ~ 10800 1750
 Wire Wire Line
-	9300 800  10250 800
-Wire Wire Line
 	10250 1100 10250 800
+Wire Wire Line
+	10250 800  10650 800
+Wire Wire Line
+	8500 800  8850 800
+$Comp
+L Device:L L?
+U 1 1 5C9C6E85
+P 9550 800
+F 0 "L?" V 9740 800 50  0000 C CNN
+F 1 "4.7nH" V 9649 800 50  0000 C CNN
+F 2 "Inductor_SMD:L_0805_2012Metric_Pad1.15x1.40mm_HandSolder" H 9550 800 50  0001 C CNN
+F 3 "~" H 9550 800 50  0001 C CNN
+	1    9550 800
+	0    -1   -1   0
+$EndComp
+$Comp
+L Device:C_Small C?
+U 1 1 5C9C8572
+P 9100 1100
+AR Path="/5C9C8572" Ref="C?"  Part="1"
+AR Path="/5C9FDFE4/5C9C8572" Ref="C?"  Part="1"
+F 0 "C?" V 8871 1100 50  0000 C CNN
+F 1 "1.0pF" V 8962 1100 50  0000 C CNN
+F 2 "Capacitor_SMD:C_0805_2012Metric_Pad1.15x1.40mm_HandSolder" H 9100 1100 50  0001 C CNN
+F 3 "~" H 9100 1100 50  0001 C CNN
+	1    9100 1100
+	0    1    1    0
+$EndComp
+Wire Wire Line
+	9150 800  9300 800
+Wire Wire Line
+	9300 800  9300 1100
+Wire Wire Line
+	9300 1100 9200 1100
+Connection ~ 9300 800
+Wire Wire Line
+	9300 800  9400 800
+Wire Wire Line
+	9000 1100 8700 1100
+Wire Wire Line
+	8700 1100 8700 1300
+Connection ~ 8700 1300
+Wire Wire Line
+	10250 800  9700 800
 Connection ~ 10250 800
-Wire Wire Line
-	10250 800  10650 800
 $EndSCHEMATC

Commit message: added basic varient
Parts:
- removed C10: nc, Capacitor_SMD:C_0805_2012Metric_Pad1.15x1.40mm_HandSolder, symbol Device:C_Small
- removed C4: 1.0uF, Capacitor_SMD:C_0805_2012Metric_Pad1.15x1.40mm_HandSolder, symbol Device:C_Small
- added C12: 0.5pf, Capacitor_SMD:C_0805_2012Metric_Pad1.15x1.40mm_HandSolder, symbol Device:C_Small
- added C13: 47nf, Capacitor_SMD:C_0805_2012Metric_Pad1.15x1.40mm_HandSolder, symbol Device:C_Small
- added C14: 100pf, Capacitor_SMD:C_0805_2012Metric_Pad1.15x1.40mm_HandSolder, symbol Device:C_Small
- added C15, C16: 12pf, Capacitor_SMD:C_0805_2012Metric_Pad1.15x1.40mm_HandSolder, symbol Device:C_Small
- added C6: 100nf, Capacitor_SMD:C_0805_2012Metric_Pad1.15x1.40mm_HandSolder, symbol Device:C_Small
- added Y1: 32mhzCrystal, Crystal:Crystal_SMD_2012-2Pin_2.0x1.2mm_HandSoldering, symbol Device:Crystal
- C1: renamed from C13; value 1.0uF -> 4.7uF
- C4: renamed from C3; value 1.0uF -> 100nf
- C5: value 1.0uF -> 100nF
- C8: renamed from C7; value 407uF -> 4.7uF
- gave numbers to parts that had none: 2
- renumbered C9 to C10, C14 to C17, C1 to C2, C2 to C3, C6 to C7, C8 to C9, L2 to L1, L1 to L2, L4 to L5
Connections:
- net labels added: 1.3vsup_decup2(rf)(dec6), VDD(AD14), VSS_BOTT, XC1, XC2, psu_decup(dec3)
- net labels removed: 1.3vsup_decup(rf)(dec2), VDD(A14)
- wire segments 75 -> 104
Other:
- moved on the sheet: C1, C10, C17, C7, C8, C9, L1

Commit message: optimized layout
Parts:
- ANT1: symbol SamacSys_Parts:CONUFL001-SMD -> hat-rescue:CONUFL001-SMD-SamacSys_Parts
Changed lines of the file:
@@
 EESchema Schematic File Version 4
 LIBS:hat-cache
-EELAYER 26 0
+EELAYER 29 0
 EELAYER END
 $Descr A4 11693 8268
@@
 	11100 1750 11100 1800
 $Comp
-L SamacSys_Parts:CONUFL001-SMD ANT1
+L hat-rescue:CONUFL001-SMD-SamacSys_Parts ANT1
 U 1 1 5C885D44
 P 10250 1100
+AR Path="/5C885D44" Ref="ANT1"  Part="1"
+AR Path="/5C9FDFE4/5C885D44" Ref="ANT1"  Part="1"
 F 0 "ANT1" H 10850 1365 50  0000 C CNN
 F 1 "CONUFL001-SMD" H 10850 1274 50  0000 C CNN
